File: keyboard-pcb.kicad_pcb (KiCad board)
At the start: 2 copper layers, 352.6 x 204 mm, 361 parts, among them J1 Conn_01x05, J2 USB_C_Receptacle_USB2.0_16P, SW1 BOOT, SW2 RESET, U1 STM32F072CBTx, U2 74AHCT1G125, U3 XC6206PxxxMR

Commit message: usb and ldo routing
Parts:
- C90: value 1uF -> 10uF
- D1, F1, J2, R1, R2, R3, R4, R5, SW1, SW2, U2, U3: moved to B.Cu
- moved U2 213.7 mm to (330.7, 38.9), turned to 180 degrees
- moved D1 212.7 mm to (323.2, 35.8), turned to 180 degrees
- moved F1 212.4 mm to (310.3, 27.4), turned to 180 degrees
- moved R4 202.2 mm to (329.1, 28.1), turned to 90 degrees
- moved R5 197.8 mm to (317.4, 28.1), turned to -90 degrees
- moved R3 189.6 mm to (329.4, 41.7), turned to -90 degrees
- moved J1 179.0 mm to (192.8, 26.7), turned to 90 degrees
- moved C94 177.8 mm to (333.9, 43.2)
- moved C91 127.8 mm to (129.3, 136.4)
- moved R1 108.2 mm to (129.8, 128.4), turned to 180 degrees
- moved R2 107.2 mm to (129.8, 132.2), turned to 180 degrees
- moved SW1 102.2 mm to (121.4, 128.8), turned to 180 degrees
- moved SW2 102.2 mm to (121.4, 135.8), turned to 180 degrees
- moved C93 95.6 mm to (182.6, 131.8)
- moved C92 93.6 mm to (185.2, 127.9)
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Connections:
- D1 pad 2: D- -> D+
- D1 pad 3: D+ -> D-
- R4 pad 1: GND -> Net-(J2-CC2)
- R4 pad 2: Net-(J2-CC2) -> GND
- R5 pad 1: Net-(J2-CC1) -> GND
- R5 pad 2: GND -> Net-(J2-CC1)
Routing:
- net +5V: track 0.00 -> 246.9 mm, vias 0 -> 4
- net D+: track 0.00 -> 239.1 mm, vias 0 -> 2
- net D-: track 0.00 -> 238.4 mm, vias 0 -> 2
- net +3V3: track 0.00 -> 44.2 mm, vias 0 -> 2
- net col6: track 86.1 -> 126.3 mm, vias 0 -> 1
- net VBUS: track 0.00 -> 26.5 mm
- net GND: track 0.00 -> 24.7 mm
- net col14: track 219.0 -> 241.4 mm, vias 1 -> 3
- net col7: track 86.1 -> 107.5 mm, vias 0 -> 1
- net col12: track 194.8 -> 214.9 mm
- net col13: track 201.3 -> 221.2 mm
- net Net-(J2-CC2): track 0.00 -> 10.6 mm, vias 0 -> 2
- net Net-(J2-CC1): track 0.00 -> 10.4 mm, vias 0 -> 2
- net col3: track 209.4 -> 207.2 mm
- net col4: track 189.1 -> 187.0 mm
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
Commit message: completed pcb design
Parts:
- removed S1, S2: MX_stab, PCM_marbastlib-mx:STAB_MX_2.25u
- removed S3: MX_stab, PCM_marbastlib-mx:STAB_MX_6.25u
- added H1: MountingHole_Pad, MountingHole:MountingHole_3.2mm_M3_DIN965_Pad, F.Cu at (61.1, 49.2)
- added H2: MountingHole_Pad, MountingHole:MountingHole_3.2mm_M3_DIN965_Pad, F.Cu at (61.1, 168.3)
- added H3: MountingHole_Pad, MountingHole:MountingHole_3.2mm_M3_DIN965_Pad, F.Cu at (370.7, 168.3)
- added H4: MountingHole_Pad, MountingHole:MountingHole_3.2mm_M3_DIN965_Pad, F.Cu at (370.7, 49.2)
- added H5: MountingHole_Pad, MountingHole:MountingHole_3.2mm_M3_DIN965_Pad, F.Cu at (215.9, 48.4)
- C1, C10, C11, C12, C13, C14, C15, C16, C17, C18, C19, C2, C20, C21, C22, C23, C24, C25, C26, C27, C28, C29, C3, C30, C31, C32, C33, C34, C35, C36, C37, C38, C39, C4, C40, C41, C42, C43, C44, C45, C46, C47, C48, C49, C5, C50, C51, C52, C53, C54, C55, C56, C57, C58, C59, C6, C60, C61, C62, C63, C64, C65, C66, C67, C68, C69, C7, C70, C71, C72, C73, C74, C75, C76, C77, C78, C79, C8, C80, C81, C82, C83, C84, C85, C86, C87, C88, C89, C9, C91, C94: footprint Capacitor_SMD:C_0402_1005Metric -> smd_silkscreen:C_0402_1005Metric
- LED1, LED10, LED11, LED12, LED13, LED14, LED15, LED2, LED3, LED31, LED32, LED33, LED34, LED35, LED36, LED37, LED38, LED39, LED4, LED40, LED41, LED42, LED43, LED44, LED45, LED5, LED6, LED60, LED61, LED62, LED63, LED64, LED65, LED66, LED67, LED68, LED69, LED7, LED70, LED71, LED72, LED73, LED8, LED84, LED9: value SK6812MINI-E -> MX_SK6812MINI-E; footprint LED_SMD:LED_SK6812MINI-E_3.2x2.8mm_P1.5mm_ReverseMount -> PCM_marbastlib-mx:LED_MX_6028R-ROT
- LED16, LED17, LED18, LED19, LED20, LED21, LED22, LED23, LED24, LED25, LED26, LED27, LED28, LED29, LED30, LED46, LED47, LED48, LED49, LED50, LED51, LED52, LED53, LED54, LED55, LED56, LED57, LED58, LED59, LED74, LED75, LED76, LED77, LED78, LED79, LED80, LED81, LED82, LED83: value SK6812MINI-E -> MX_SK6812MINI-E; footprint LED_SMD:LED_SK6812MINI-E_3.2x2.8mm_P1.5mm_ReverseMount -> PCM_marbastlib-mx:LED_MX_6028R
- MX1, MX10, MX11, MX12, MX13, MX14, MX15, MX16, MX17, MX18, MX19, MX2, MX20, MX21, MX22, MX23, MX24, MX25, MX26, MX27, MX28, MX29, MX3, MX30, MX32, MX33, MX34, MX35, MX36, MX37, MX38, MX39, MX4, MX40, MX41, MX42, MX43, MX44, MX45, MX47, MX48, MX49, MX5, MX50, MX51, MX52, MX53, MX54, MX55, MX56, MX57, MX59, MX6, MX61, MX62, MX63, MX64, MX65, MX66, MX67, MX68, MX69, MX7, MX70, MX71, MX72, MX73, MX78, MX79, MX8, MX80, MX81, MX82, MX83, MX9: footprint PCM_marbastlib-mx:SW_MX_HS_CPG151101S11_1u -> MX_Hotswap:MX-Hotswap-1U
- MX31: footprint PCM_marbastlib-mx:SW_MX_HS_CPG151101S11_1.5u -> MX_Hotswap:MX-Hotswap-1.5U
- MX46: footprint PCM_marbastlib-mx:SW_MX_HS_CPG151101S11_1.75u -> MX_Hotswap:MX-Hotswap-1.75U
- MX58, MX60: footprint PCM_marbastlib-mx:SW_MX_HS_CPG151101S11_1u -> MX_Hotswap:MX-Hotswap-2.25U
- MX74, MX75, MX76: footprint PCM_marbastlib-mx:SW_MX_HS_CPG151101S11_1.25u -> MX_Hotswap:MX-Hotswap-1.25U
- MX77: footprint PCM_marbastlib-mx:SW_MX_HS_CPG151101S11_1u -> MX_Hotswap:MX-Hotswap-6.25U
- R1, R2, R3, R4, R5: footprint Resistor_SMD:R_0402_1005Metric -> smd_silkscreen:R_0402_1005Metric
- moved C94 271.1 mm to (64.1, 70.3), turned to -90 degrees
- moved U2 270.7 mm to (61.8, 70.9), turned to 90 degrees
- moved R3 269.8 mm to (61.0, 67.9), turned to 90 degrees
- moved J1 153.8 mm to (250.2, 169.3), turned to -90 degrees
- moved RST1 58.7 mm to (177.7, 152.5), turned to 90 degrees
- moved C91 52.7 mm to (177.7, 157.3)
- moved C90 46.4 mm to (219.4, 163.4), turned to 0 degrees
- moved C93 46.2 mm to (217.8, 161.7)
- moved U3 46.2 mm to (221.1, 160.6)
- moved C92 46.2 mm to (220.3, 157.8)
- moved D14 42.4 mm to (309.3, 61.1)
- moved D15 42.4 mm to (328.3, 61.1)
- moved D22 42.4 mm to (175.9, 80.2)
- moved D24 42.4 mm to (214.0, 80.2)
- moved D29 42.4 mm to (309.3, 80.2)
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- renumbered SW1 to BOOT1, SW2 to RST1
Connections:
- J1 pad 4: RST -> NRST
- LED1 pad 1: GND -> +5V
- LED1 pad 2: LED_5 -> Net-(LED1-DOUT)
- LED1 pad 3: +5V -> LED_5
- LED1 pad 4: Net-(LED1-DOUT) -> GND
- LED10 pad 1: GND -> +5V
- LED10 pad 2: Net-(LED10-DIN) -> Net-(LED10-DOUT)
- LED10 pad 3: +5V -> Net-(LED10-DIN)
- LED10 pad 4: Net-(LED10-DOUT) -> GND
- LED11 pad 1: GND -> +5V
- LED11 pad 2: Net-(LED10-DOUT) -> Net-(LED11-DOUT)
- LED11 pad 3: +5V -> Net-(LED10-DOUT)
- LED11 pad 4: Net-(LED11-DOUT) -> GND
- LED12 pad 1: GND -> +5V
- LED12 pad 2: Net-(LED11-DOUT) -> Net-(LED12-DOUT)
- LED12 pad 3: +5V -> Net-(LED11-DOUT)
- LED12 pad 4: Net-(LED12-DOUT) -> GND
- LED13 pad 1: GND -> +5V
- LED13 pad 2: Net-(LED12-DOUT) -> Net-(LED13-DOUT)
- LED13 pad 3: +5V -> Net-(LED12-DOUT)
- LED13 pad 4: Net-(LED13-DOUT) -> GND
- LED14 pad 1: GND -> +5V
- LED14 pad 2: Net-(LED13-DOUT) -> Net-(LED14-DOUT)
- LED14 pad 3: +5V -> Net-(LED13-DOUT)
- LED14 pad 4: Net-(LED14-DOUT) -> GND
- LED15 pad 1: GND -> +5V
- LED15 pad 2: Net-(LED14-DOUT) -> Net-(LED15-DOUT)
- LED15 pad 3: +5V -> Net-(LED14-DOUT)
- LED15 pad 4: Net-(LED15-DOUT) -> GND
- LED16 pad 1: GND -> +5V
- LED16 pad 2: Net-(LED16-DIN) -> Net-(LED16-DOUT)
- LED16 pad 3: +5V -> Net-(LED16-DIN)
- LED16 pad 4: Net-(LED16-DOUT) -> GND
- LED17 pad 1: GND -> +5V
- LED17 pad 2: Net-(LED16-DOUT) -> Net-(LED16-DIN)
- LED17 pad 3: +5V -> Net-(LED17-DIN)
- LED17 pad 4: Net-(LED17-DOUT) -> GND
- LED18 pad 1: GND -> +5V
- LED18 pad 2: Net-(LED17-DOUT) -> Net-(LED17-DIN)
- LED18 pad 3: +5V -> Net-(LED18-DIN)
- LED18 pad 4: Net-(LED18-DOUT) -> GND
- LED19 pad 1: GND -> +5V
- LED19 pad 2: Net-(LED18-DOUT) -> Net-(LED18-DIN)
- LED19 pad 3: +5V -> Net-(LED19-DIN)
- LED19 pad 4: Net-(LED19-DOUT) -> GND
- LED2 pad 1: GND -> +5V
- LED2 pad 2: Net-(LED1-DOUT) -> Net-(LED2-DOUT)
- LED2 pad 3: +5V -> Net-(LED1-DOUT)
- LED2 pad 4: Net-(LED2-DOUT) -> GND
- LED20 pad 1: GND -> +5V
- LED20 pad 2: Net-(LED19-DOUT) -> Net-(LED19-DIN)
- LED20 pad 3: +5V -> Net-(LED20-DIN)
- LED20 pad 4: Net-(LED20-DOUT) -> GND
- LED21 pad 1: GND -> +5V
- LED21 pad 2: Net-(LED20-DOUT) -> Net-(LED20-DIN)
- LED21 pad 3: +5V -> Net-(LED21-DIN)
- LED21 pad 4: Net-(LED21-DOUT) -> GND
- LED22 pad 1: GND -> +5V
- LED22 pad 2: Net-(LED21-DOUT) -> Net-(LED21-DIN)
- LED22 pad 3: +5V -> Net-(LED22-DIN)
- LED22 pad 4: Net-(LED22-DOUT) -> GND
- LED23 pad 1: GND -> +5V
- LED23 pad 2: Net-(LED22-DOUT) -> Net-(LED22-DIN)
- LED23 pad 3: +5V -> Net-(LED23-DIN)
- LED23 pad 4: Net-(LED23-DOUT) -> GND
- LED24 pad 1: GND -> +5V
- LED24 pad 2: Net-(LED23-DOUT) -> Net-(LED23-DIN)
- LED24 pad 3: +5V -> Net-(LED24-DIN)
- LED24 pad 4: Net-(LED24-DOUT) -> GND
- LED25 pad 1: GND -> +5V
- LED25 pad 2: Net-(LED24-DOUT) -> Net-(LED24-DIN)
- LED25 pad 3: +5V -> Net-(LED25-DIN)
- LED25 pad 4: Net-(LED25-DOUT) -> GND
- LED26 pad 1: GND -> +5V
- LED26 pad 2: Net-(LED25-DOUT) -> Net-(LED25-DIN)
- LED26 pad 3: +5V -> Net-(LED26-DIN)
- LED26 pad 4: Net-(LED26-DOUT) -> GND
- LED27 pad 1: GND -> +5V
- LED27 pad 2: Net-(LED26-DOUT) -> Net-(LED26-DIN)
- LED27 pad 3: +5V -> Net-(LED27-DIN)
- LED27 pad 4: Net-(LED27-DOUT) -> GND
- LED28 pad 1: GND -> +5V
- LED28 pad 2: Net-(LED27-DOUT) -> Net-(LED27-DIN)
- LED28 pad 3: +5V -> Net-(LED28-DIN)
- LED28 pad 4: Net-(LED28-DOUT) -> GND
- LED29 pad 1: GND -> +5V
- LED29 pad 2: Net-(LED28-DOUT) -> Net-(LED28-DIN)
- LED29 pad 3: +5V -> Net-(LED29-DIN)
- LED29 pad 4: Net-(LED29-DOUT) -> GND
- LED3 pad 1: GND -> +5V
- LED3 pad 2: Net-(LED2-DOUT) -> Net-(LED3-DOUT)
- LED3 pad 3: +5V -> Net-(LED2-DOUT)
- LED3 pad 4: Net-(LED3-DOUT) -> GND
- LED30 pad 1: GND -> +5V
- LED30 pad 2: Net-(LED29-DOUT) -> Net-(LED29-DIN)
- LED30 pad 3: +5V -> Net-(LED30-DIN)
- LED30 pad 4: Net-(LED30-DOUT) -> GND
- LED31 pad 1: GND -> +5V
- LED31 pad 2: Net-(LED30-DOUT) -> Net-(LED31-DOUT)
- LED31 pad 3: +5V -> Net-(LED16-DOUT)
- LED31 pad 4: Net-(LED31-DOUT) -> GND
- LED32 pad 1: GND -> +5V
- LED32 pad 2: Net-(LED31-DOUT) -> Net-(LED32-DOUT)
- LED32 pad 3: +5V -> Net-(LED31-DOUT)
- LED32 pad 4: Net-(LED32-DOUT) -> GND
- LED33 pad 1: GND -> +5V
- LED33 pad 2: Net-(LED32-DOUT) -> Net-(LED33-DOUT)
- LED33 pad 3: +5V -> Net-(LED32-DOUT)
- LED33 pad 4: Net-(LED33-DOUT) -> GND
- LED34 pad 1: GND -> +5V
- LED34 pad 2: Net-(LED33-DOUT) -> Net-(LED34-DOUT)
- LED34 pad 3: +5V -> Net-(LED33-DOUT)
- LED34 pad 4: Net-(LED34-DOUT) -> GND
- LED35 pad 1: GND -> +5V
- LED35 pad 2: Net-(LED34-DOUT) -> Net-(LED35-DOUT)
- LED35 pad 3: +5V -> Net-(LED34-DOUT)
- LED35 pad 4: Net-(LED35-DOUT) -> GND
- LED36 pad 1: GND -> +5V
- LED36 pad 2: Net-(LED35-DOUT) -> Net-(LED36-DOUT)
- LED36 pad 3: +5V -> Net-(LED35-DOUT)
- LED36 pad 4: Net-(LED36-DOUT) -> GND
- LED37 pad 1: GND -> +5V
- LED37 pad 2: Net-(LED36-DOUT) -> Net-(LED37-DOUT)
- LED37 pad 3: +5V -> Net-(LED36-DOUT)
- LED37 pad 4: Net-(LED37-DOUT) -> GND
- LED38 pad 1: GND -> +5V
- LED38 pad 2: Net-(LED37-DOUT) -> Net-(LED38-DOUT)
- LED38 pad 3: +5V -> Net-(LED37-DOUT)
- LED38 pad 4: Net-(LED38-DOUT) -> GND
- LED39 pad 1: GND -> +5V
- LED39 pad 2: Net-(LED38-DOUT) -> Net-(LED39-DOUT)
- LED39 pad 3: +5V -> Net-(LED38-DOUT)
- LED39 pad 4: Net-(LED39-DOUT) -> GND
- LED4 pad 1: GND -> +5V
- LED4 pad 2: Net-(LED3-DOUT) -> Net-(LED4-DOUT)
- LED4 pad 3: +5V -> Net-(LED3-DOUT)
- LED4 pad 4: Net-(LED4-DOUT) -> GND
- LED40 pad 1: GND -> +5V
- LED40 pad 2: Net-(LED39-DOUT) -> Net-(LED40-DOUT)
- LED40 pad 3: +5V -> Net-(LED39-DOUT)
- LED40 pad 4: Net-(LED40-DOUT) -> GND
- LED41 pad 1: GND -> +5V
- LED41 pad 2: Net-(LED40-DOUT) -> Net-(LED41-DOUT)
- LED41 pad 3: +5V -> Net-(LED40-DOUT)
- LED41 pad 4: Net-(LED41-DOUT) -> GND
- LED42 pad 1: GND -> +5V
- LED42 pad 2: Net-(LED41-DOUT) -> Net-(LED42-DOUT)
- LED42 pad 3: +5V -> Net-(LED41-DOUT)
- LED42 pad 4: Net-(LED42-DOUT) -> GND
- LED43 pad 1: GND -> +5V
- LED43 pad 2: Net-(LED42-DOUT) -> Net-(LED43-DOUT)
- LED43 pad 3: +5V -> Net-(LED42-DOUT)
- LED43 pad 4: Net-(LED43-DOUT) -> GND
- LED44 pad 1: GND -> +5V
- LED44 pad 2: Net-(LED43-DOUT) -> Net-(LED44-DOUT)
- LED44 pad 3: +5V -> Net-(LED43-DOUT)
- LED44 pad 4: Net-(LED44-DOUT) -> GND
- LED45 pad 1: GND -> +5V
- LED45 pad 2: Net-(LED44-DOUT) -> Net-(LED45-DOUT)
- LED45 pad 3: +5V -> Net-(LED44-DOUT)
- LED45 pad 4: Net-(LED45-DOUT) -> GND
- LED46 pad 1: GND -> +5V
- LED46 pad 2: Net-(LED45-DOUT) -> Net-(LED46-DOUT)
- LED46 pad 3: +5V -> Net-(LED46-DIN)
- LED46 pad 4: Net-(LED46-DOUT) -> GND
- LED47 pad 1: GND -> +5V
- LED47 pad 2: Net-(LED46-DOUT) -> Net-(LED46-DIN)
- LED47 pad 3: +5V -> Net-(LED47-DIN)
- LED47 pad 4: Net-(LED47-DOUT) -> GND
- LED48 pad 1: GND -> +5V
- LED48 pad 2: Net-(LED47-DOUT) -> Net-(LED47-DIN)
- LED48 pad 3: +5V -> Net-(LED48-DIN)
- LED48 pad 4: Net-(LED48-DOUT) -> GND
- LED49 pad 1: GND -> +5V
- LED49 pad 2: Net-(LED48-DOUT) -> Net-(LED48-DIN)
- LED49 pad 3: +5V -> Net-(LED49-DIN)
- LED49 pad 4: Net-(LED49-DOUT) -> GND
- LED5 pad 1: GND -> +5V
- LED5 pad 2: Net-(LED4-DOUT) -> Net-(LED5-DOUT)
- LED5 pad 3: +5V -> Net-(LED4-DOUT)
- LED5 pad 4: Net-(LED5-DOUT) -> GND
- LED50 pad 1: GND -> +5V
- LED50 pad 2: Net-(LED49-DOUT) -> Net-(LED49-DIN)
- LED50 pad 3: +5V -> Net-(LED50-DIN)
- LED50 pad 4: Net-(LED50-DOUT) -> GND
- LED51 pad 1: GND -> +5V
- LED51 pad 2: Net-(LED50-DOUT) -> Net-(LED50-DIN)
- LED51 pad 3: +5V -> Net-(LED51-DIN)
- LED51 pad 4: Net-(LED51-DOUT) -> GND
- LED52 pad 1: GND -> +5V
- LED52 pad 2: Net-(LED51-DOUT) -> Net-(LED51-DIN)
- LED52 pad 3: +5V -> Net-(LED52-DIN)
- LED52 pad 4: Net-(LED52-DOUT) -> GND
- LED53 pad 1: GND -> +5V
- LED53 pad 2: Net-(LED52-DOUT) -> Net-(LED52-DIN)
- LED53 pad 3: +5V -> Net-(LED53-DIN)
- LED53 pad 4: Net-(LED53-DOUT) -> GND
- LED54 pad 1: GND -> +5V
- LED54 pad 2: Net-(LED53-DOUT) -> Net-(LED53-DIN)
- LED54 pad 3: +5V -> Net-(LED54-DIN)
- LED54 pad 4: Net-(LED54-DOUT) -> GND
- LED55 pad 1: GND -> +5V
- LED55 pad 2: Net-(LED54-DOUT) -> Net-(LED54-DIN)
- LED55 pad 3: +5V -> Net-(LED55-DIN)
- LED55 pad 4: Net-(LED55-DOUT) -> GND
- LED56 pad 1: GND -> +5V
- LED56 pad 2: Net-(LED55-DOUT) -> Net-(LED55-DIN)
- LED56 pad 3: +5V -> Net-(LED56-DIN)
- LED56 pad 4: Net-(LED56-DOUT) -> GND
- LED57 pad 1: GND -> +5V
- LED57 pad 2: Net-(LED56-DOUT) -> Net-(LED56-DIN)
- LED57 pad 3: +5V -> Net-(LED57-DIN)
- LED57 pad 4: Net-(LED57-DOUT) -> GND
- LED58 pad 1: GND -> +5V
- LED58 pad 2: Net-(LED57-DOUT) -> Net-(LED57-DIN)
- LED58 pad 3: +5V -> Net-(LED58-DIN)
- LED58 pad 4: Net-(LED58-DOUT) -> GND
- LED59 pad 1: GND -> +5V
- LED59 pad 2: Net-(LED58-DOUT) -> Net-(LED58-DIN)
- LED59 pad 3: +5V -> Net-(LED45-DOUT)
- LED59 pad 4: Net-(LED59-DOUT) -> GND
- LED6 pad 1: GND -> +5V
- LED6 pad 2: Net-(LED5-DOUT) -> Net-(LED6-DOUT)
- LED6 pad 3: +5V -> Net-(LED5-DOUT)
- LED6 pad 4: Net-(LED6-DOUT) -> GND
- LED60 pad 1: GND -> +5V
- LED60 pad 2: Net-(LED59-DOUT) -> Net-(LED60-DOUT)
- LED60 pad 3: +5V -> Net-(LED46-DOUT)
- LED60 pad 4: Net-(LED60-DOUT) -> GND
- LED61 pad 1: GND -> +5V
- LED61 pad 2: Net-(LED60-DOUT) -> Net-(LED61-DOUT)
- LED61 pad 3: +5V -> Net-(LED60-DOUT)
- LED61 pad 4: Net-(LED61-DOUT) -> GND
- LED62 pad 1: GND -> +5V
- LED62 pad 2: Net-(LED61-DOUT) -> Net-(LED62-DOUT)
- LED62 pad 3: +5V -> Net-(LED61-DOUT)
- LED62 pad 4: Net-(LED62-DOUT) -> GND
- LED63 pad 1: GND -> +5V
- LED63 pad 2: Net-(LED62-DOUT) -> Net-(LED63-DOUT)
- LED63 pad 3: +5V -> Net-(LED62-DOUT)
- LED63 pad 4: Net-(LED63-DOUT) -> GND
- LED64 pad 1: GND -> +5V
- LED64 pad 2: Net-(LED63-DOUT) -> Net-(LED64-DOUT)
- LED64 pad 3: +5V -> Net-(LED63-DOUT)
- LED64 pad 4: Net-(LED64-DOUT) -> GND
- LED65 pad 1: GND -> +5V
- LED65 pad 2: Net-(LED64-DOUT) -> Net-(LED65-DOUT)
- LED65 pad 3: +5V -> Net-(LED64-DOUT)
- LED65 pad 4: Net-(LED65-DOUT) -> GND
- LED66 pad 1: GND -> +5V
- LED66 pad 2: Net-(LED65-DOUT) -> Net-(LED66-DOUT)
- LED66 pad 3: +5V -> Net-(LED65-DOUT)
- LED66 pad 4: Net-(LED66-DOUT) -> GND
- LED67 pad 1: GND -> +5V
- LED67 pad 2: Net-(LED66-DOUT) -> Net-(LED67-DOUT)
- LED67 pad 3: +5V -> Net-(LED66-DOUT)
- LED67 pad 4: Net-(LED67-DOUT) -> GND
- LED68 pad 1: GND -> +5V
- LED68 pad 2: Net-(LED67-DOUT) -> Net-(LED68-DOUT)
- LED68 pad 3: +5V -> Net-(LED67-DOUT)
- LED68 pad 4: Net-(LED68-DOUT) -> GND
- LED69 pad 1: GND -> +5V
- LED69 pad 2: Net-(LED68-DOUT) -> Net-(LED69-DOUT)
- LED69 pad 3: +5V -> Net-(LED68-DOUT)
- LED69 pad 4: Net-(LED69-DOUT) -> GND
- LED7 pad 1: GND -> +5V
- LED7 pad 2: Net-(LED6-DOUT) -> Net-(LED7-DOUT)
- LED7 pad 3: +5V -> Net-(LED6-DOUT)
- LED7 pad 4: Net-(LED7-DOUT) -> GND
- LED70 pad 1: GND -> +5V
- LED70 pad 2: Net-(LED69-DOUT) -> Net-(LED70-DOUT)
- LED70 pad 3: +5V -> Net-(LED69-DOUT)
- LED70 pad 4: Net-(LED70-DOUT) -> GND
- LED71 pad 1: GND -> +5V
- LED71 pad 2: Net-(LED70-DOUT) -> Net-(LED71-DOUT)
- LED71 pad 3: +5V -> Net-(LED70-DOUT)
- LED71 pad 4: Net-(LED71-DOUT) -> GND
- LED72 pad 1: GND -> +5V
- LED72 pad 2: Net-(LED71-DOUT) -> Net-(LED72-DOUT)
- LED72 pad 3: +5V -> Net-(LED71-DOUT)
- LED72 pad 4: Net-(LED72-DOUT) -> GND
- LED73 pad 1: GND -> +5V
- LED73 pad 2: Net-(LED72-DOUT) -> Net-(LED73-DOUT)
- LED73 pad 3: +5V -> Net-(LED72-DOUT)
- LED73 pad 4: Net-(LED73-DOUT) -> GND
- LED74 pad 1: GND -> +5V
- LED74 pad 2: Net-(LED73-DOUT) -> unconnected-(LED74-DOUT-Pad2)
- LED74 pad 3: +5V -> Net-(LED74-DIN)
- LED74 pad 4: Net-(LED74-DOUT) -> GND
- LED75 pad 1: GND -> +5V
- LED75 pad 2: Net-(LED74-DOUT) -> Net-(LED74-DIN)
- LED75 pad 3: +5V -> Net-(LED75-DIN)
- LED75 pad 4: Net-(LED75-DOUT) -> GND
- LED76 pad 1: GND -> +5V
- LED76 pad 2: Net-(LED75-DOUT) -> Net-(LED75-DIN)
- LED76 pad 3: +5V -> Net-(LED76-DIN)
- LED76 pad 4: Net-(LED76-DOUT) -> GND
- LED77 pad 1: GND -> +5V
- LED77 pad 2: Net-(LED76-DOUT) -> Net-(LED76-DIN)
- LED77 pad 3: +5V -> Net-(LED77-DIN)
- LED77 pad 4: Net-(LED77-DOUT) -> GND
- LED78 pad 1: GND -> +5V
- LED78 pad 2: Net-(LED77-DOUT) -> Net-(LED77-DIN)
- LED78 pad 3: +5V -> Net-(LED78-DIN)
- LED78 pad 4: Net-(LED78-DOUT) -> GND
- LED79 pad 1: GND -> +5V
- LED79 pad 2: Net-(LED78-DOUT) -> Net-(LED78-DIN)
- LED79 pad 3: +5V -> Net-(LED79-DIN)
- LED79 pad 4: Net-(LED79-DOUT) -> GND
- LED8 pad 1: GND -> +5V
- LED8 pad 2: Net-(LED7-DOUT) -> Net-(LED8-DOUT)
- LED8 pad 3: +5V -> Net-(LED7-DOUT)
- LED8 pad 4: Net-(LED8-DOUT) -> GND
- LED80 pad 1: GND -> +5V
- LED80 pad 2: Net-(LED79-DOUT) -> Net-(LED79-DIN)
- LED80 pad 3: +5V -> Net-(LED80-DIN)
- LED80 pad 4: Net-(LED80-DOUT) -> GND
- LED81 pad 1: GND -> +5V
- LED81 pad 2: Net-(LED80-DOUT) -> Net-(LED80-DIN)
- LED81 pad 3: +5V -> Net-(LED81-DIN)
- LED81 pad 4: Net-(LED81-DOUT) -> GND
- LED82 pad 1: GND -> +5V
- LED82 pad 2: Net-(LED81-DOUT) -> Net-(LED81-DIN)
- LED82 pad 3: +5V -> Net-(LED82-DIN)
- LED82 pad 4: Net-(LED82-DOUT) -> GND
- LED83 pad 1: GND -> +5V
- LED83 pad 2: Net-(LED82-DOUT) -> Net-(LED82-DIN)
- LED83 pad 3: +5V -> Net-(LED73-DOUT)
- LED83 pad 4: unconnected-(LED83-DOUT-Pad4) -> GND
- LED84 pad 1: GND -> +5V
- LED84 pad 2: Net-(LED15-DOUT) -> Net-(LED30-DIN)
- LED84 pad 3: +5V -> Net-(LED15-DOUT)
- LED84 pad 4: Net-(LED16-DIN) -> GND
- LED9 pad 1: GND -> +5V
- LED9 pad 2: Net-(LED8-DOUT) -> Net-(LED10-DIN)
- LED9 pad 3: +5V -> Net-(LED8-DOUT)
- LED9 pad 4: Net-(LED10-DIN) -> GND
- U1 pad 11: unconnected-(U1-PA1-Pad11) -> col6
- U1 pad 12: unconnected-(U1-PA2-Pad12) -> col7
- U1 pad 13: col6 -> unconnected-(U1-PA3-Pad13)
- U1 pad 14: col7 -> unconnected-(U1-PA4-Pad14)
- U1 pad 17: unconnected-(U1-PA7-Pad17) -> row0
- U1 pad 18: unconnected-(U1-PB0-Pad18) -> row1
- U1 pad 19: unconnected-(U1-PB1-Pad19) -> row2
- U1 pad 20: unconnected-(U1-PB2-Pad20) -> row3
- U1 pad 21: unconnected-(U1-PB10-Pad21) -> row5
- U1 pad 22: unconnected-(U1-PB11-Pad22) -> row4
- U1 pad 45: unconnected-(U1-PB8-Pad45) -> LED_3v3
Routing:
- net +5V: track 246.9 -> 2076.2 mm, vias 4 -> 11
- net LED_3v3: track 0.00 -> 271.5 mm, vias 0 -> 4
- net row2: track 269.8 -> 488.0 mm, vias 0 -> 2
- net row4: track 262.7 -> 449.9 mm, vias 0 -> 4
- net row3: track 286.4 -> 448.9 mm, vias 0 -> 2
- net row0: track 275.1 -> 385.7 mm, vias 0 -> 2
- net row1: track 265.0 -> 373.4 mm, vias 0 -> 2
- net +3V3: track 44.2 -> 151.1 mm, vias 2 -> 7
- net BOOT: track 0.00 -> 102.2 mm, vias 0 -> 2
- net NRST: track 0.00 -> 100.6 mm, vias 0 -> 5
- net Net-(LED77-DIN): track 0.00 -> 80.2 mm, vias 0 -> 4
- net col0: track 288.9 -> 364.7 mm, vias 1 -> 7
- net Net-(LED76-DIN): track 0.00 -> 66.6 mm
- net GND: track 24.7 -> 68.7 mm, vias 0 -> 73
- net row5: track 307.3 -> 345.1 mm, vias 4 -> 3
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- added copper zone on B.Cu, net GND
- added copper zone on F.Cu, net GND
Other:
- board size 352.6 x 204 mm -> 317.5 x 127 mm
