File: keyboard-pcb.kicad_pcb (KiCad board)
At the start: 2 copper layers, 317.5 x 127 mm, 363 parts, among them J1 Conn_01x05, J2 USB_C_Receptacle_USB2.0_16P, U1 STM32F072CBTx, U2 74AHCT1G125, U3 XC6206PxxxMR

Commit message: small edge cut changes
Parts:
- moved J2 1.59 mm to (358.3, 48.6)
Routing:
- net D-: track 240.7 -> 243.8 mm
- net GND: track 68.7 -> 71.8 mm
- net VBUS: track 26.5 -> 28.1 mm
- net Net-(J2-CC2): track 10.2 -> 11.7 mm
- net Net-(J2-CC1): track 10.4 -> 12.0 mm
- net D+: track 241.4 -> 243.0 mm
Other:
- outline, holes or cut-outs redrawn
Changed lines of the file:
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@@
 	(footprint "PCM_marbastlib-various:USB_C_Receptacle_HRO_TYPE-C-31-M-12"
 		(layer "B.Cu")
-		(at 358.267091 50.2031)
+		(at 358.267091 48.6156)
 		(descr "USB Type-C receptacle for USB 2.0 and PD, http://www.krhro.com/uploads/soft/180320/1-1P320120243.pdf")
 		(tags "usb usb-c 2.0 pd")
@@
 		)
 	)
-	(gr_rect
-		(start 57.15 45.24375)
-		(end 374.65 172.24375)
+	(gr_arc
+		(start 57.15 49.24375)
+		(mid 58.321591 46.415355)
+		(end 61.15 45.24375)
+		(stroke
+			(width 0.05)
+			(type default)
+		)
+		(layer "Edge.Cuts")
+	)
+	(gr_line
+		(start 57.15 168.24375)
+		(end 57.15 49.24375)
+		(stroke
+			(width 0.05)
+			(type default)
+		)
+		(layer "Edge.Cuts")
+	)
+	(gr_line
+		(start 61.15 45.24375)
+		(end 370.65 45.24375)
+		(stroke
+			(width 0.05)
+			(type default)
+		)
+		(layer "Edge.Cuts")
+	)
+	(gr_arc
+		(start 61.15 172.24375)
+		(mid 58.321573 171.072177)
+		(end 57.15 168.24375)
+		(stroke
+			(width 0.05)
+			(type default)
+		)
+		(layer "Edge.Cuts")
+	)
+	(gr_arc
+		(start 370.65 45.24375)
+		(mid 373.478427 46.415323)
+		(end 374.65 49.24375)
+		(stroke
+			(width 0.05)
+			(type default)
+		)
+		(layer "Edge.Cuts")
+	)
+	(gr_line
+		(start 370.65 172.24375)
+		(end 61.15 172.24375)
+		(stroke
+			(width 0.05)
+			(type default)
+		)
+		(layer "Edge.Cuts")
+	)
+	(gr_line
+		(start 374.65 49.24375)
+		(end 374.65 168.24375)
+		(stroke
+			(width 0.05)
+			(type default)
+		)
+		(layer "Edge.Cuts")
+	)
+	(gr_arc
+		(start 374.65 168.24375)
+		(mid 373.478409 171.072145)
+		(end 370.65 172.24375)
 		(stroke
 			(width 0.05)
 			(type default)
 		)
-		(fill no)
 		(layer "Edge.Cuts")
 	)
@@
 	)
 	(segment
-		(start 361.517091 54.2481)
-		(end 361.672091 54.2481)
-		(width 0.381)
-		(layer "B.Cu")
-		(net "GND")
-	)
-	(segment
-		(start 353.947091 53.3331)
-		(end 354.102091 53.3331)
+		(start 354.102091 51.7456)
+		(end 355.017091 52.6606)
 		(width 0.381)
 		(layer "B.Cu")
@@
 	)
 	(segment
-		(start 353.474091 55.7911)
-		(end 355.017091 54.2481)
+		(start 361.517091 55.8391)
+		(end 361.517091 52.6606)
 		(width 0.381)
 		(layer "B.Cu")
@@
 	)
 	(segment
-		(start 353.947091 49.1531)
-		(end 362.587091 49.1531)
+		(start 353.947091 47.5656)
+		(end 362.587091 47.5656)
+		(width 0.381)
+		(layer "B.Cu")
+		(net "GND")
+	)
+	(segment
+		(start 353.947091 51.7456)
+		(end 354.102091 51.7456)
 		(width 0.381)
 		(layer "B.Cu")
@@
 	)
 	(segment
-		(start 175.778091 155.6131)
-		(end 175.778091 149.3131)
+		(start 355.017091 52.6606)
+		(end 355.017091 54.2481)
 		(width 0.381)
 		(layer "B.Cu")
@@
 	)
 	(segment
-		(start 353.947091 53.3331)
-		(end 353.947091 49.1531)
+		(start 175.778091 155.6131)
+		(end 175.778091 149.3131)
 		(width 0.381)
 		(layer "B.Cu")
@@
 	)
 	(segment
-		(start 354.102091 53.3331)
-		(end 355.017091 54.2481)
+		(start 353.947091 51.7456)
+		(end 353.947091 47.5656)
 		(width 0.381)
 		(layer "B.Cu")
@@
 	)
 	(segment
-		(start 62.799091 71.379101)
-		(end 62.799091 72.0416)
+		(start 362.432091 51.7456)
+		(end 361.517091 52.6606)
 		(width 0.381)
 		(layer "B.Cu")
@@
 	)
 	(segment
-		(start 361.672091 54.2481)
-		(end 362.587091 53.3331)
+		(start 62.799091 71.379101)
+		(end 62.799091 72.0416)
 		(width 0.381)
 		(layer "B.Cu")
@@
 	)
 	(segment
-		(start 361.517091 55.8391)
-		(end 361.517091 54.2481)
+		(start 362.587091 51.7456)
+		(end 362.432091 51.7456)
+		(width 0.381)
+		(layer "B.Cu")
+		(net "GND")
+	)
+	(segment
+		(start 355.017091 54.2481)
+		(end 353.474091 55.7911)
 		(width 0.381)
 		(layer "B.Cu")
@@
 	)
 	(segment
-		(start 362.587091 53.3331)
-		(end 362.587091 49.1531)
+		(start 362.587091 51.7456)
+		(end 362.587091 47.5656)
 		(width 0.381)
 		(layer "B.Cu")
@@
 	)
 	(segment
-		(start 357.517091 54.2481)
-		(end 357.517091 55.6761)
-		(width 0.254)
-		(layer "B.Cu")
-		(net "D-")
-	)
-	(segment
-		(start 358.517091 54.2481)
-		(end 358.517091 55.6681)
+		(start 358.517091 55.6681)
+		(end 358.517091 52.6606)
 		(width 0.254)
 		(layer "B.Cu")
@@
 	)
 	(segment
+		(start 357.517091 55.6761)
+		(end 357.517091 52.6606)
+		(width 0.254)
+		(layer "B.Cu")
+		(net "D-")
+	)
+	(segment
 		(start 357.267091 59.7891)
 		(end 357.267091 61.961909)
@@
 	)
 	(segment
-		(start 350.11345 64.518)
-		(end 349.776238 64.518)
+		(start 358.013091 56.1721)
+		(end 357.517091 55.6761)
 		(width 0.254)
 		(layer "B.Cu")
@@
 	)
 	(segment
-		(start 358.517091 55.6681)
-		(end 358.013091 56.1721)
+		(start 350.11345 64.518)
+		(end 349.776238 64.518)
 		(width 0.254)
 		(layer "B.Cu")
@@
 	)
 	(segment
-		(start 357.517091 55.6761)
-		(end 358.013091 56.1721)
+		(start 358.013091 56.1721)
+		(end 358.517091 55.6681)
 		(width 0.254)
 		(layer "B.Cu")
@@
 	)
 	(segment
-		(start 359.017091 56.0031)
-		(end 358.467091 56.5531)
+		(start 242.576709 157.5001)
+		(end 255.518709 170.4421)
 		(width 0.254)
 		(layer "B.Cu")
@@
 	)
 	(segment
-		(start 359.017091 54.2481)
-		(end 359.017091 56.0031)
+		(start 359.017091 56.0031)
+		(end 359.017091 52.6606)
 		(width 0.254)
 		(layer "B.Cu")
@@
 	)
 	(segment
-		(start 242.576709 157.5001)
-		(end 255.518709 170.4421)
+		(start 358.017091 51.865008)
+		(end 358.017091 52.6606)
 		(width 0.254)
 		(layer "B.Cu")
@@
 	)
 	(segment
-		(start 358.017091 53.452508)
-		(end 358.017091 54.2481)
+		(start 238.858591 157.4981)
+		(end 238.860591 157.5001)
 		(width 0.254)
 		(layer "B.Cu")
@@
 	)
 	(segment
-		(start 238.858591 157.4981)
-		(end 238.860591 157.5001)
+		(start 358.467091 56.5531)
+		(end 359.017091 56.0031)
 		(width 0.254)
 		(layer "B.Cu")
@@
 	)
 	(segment
-		(start 358.467091 56.5531)
-		(end 358.467091 58.9891)
-		(width 0.254)
-		(layer "B.Cu")
-		(net "D+")
-	)
-	(segment
 		(start 349.257773 65.022)
 		(end 348.505091 65.774682)
@@
 	)
 	(segment
-		(start 358.760683 53.1961)
-		(end 358.273499 53.1961)
+		(start 359.267091 59.7891)
+		(end 358.467091 58.9891)
+		(width 0.254)
+		(layer "B.Cu")
+		(net "D+")
+	)
+	(segment
+		(start 358.760683 51.6086)
+		(end 358.273499 51.6086)
 		(width 0.254)
 		(layer "B.Cu")
@@
 	)
 	(segment
-		(start 359.017091 54.2481)
-		(end 359.017091 53.452508)
+		(start 359.017091 52.6606)
+		(end 359.017091 51.865008)
 		(width 0.254)
 		(layer "B.Cu")
@@
 	(segment
 		(start 358.467091 58.9891)
-		(end 359.267091 59.7891)
+		(end 358.467091 56.5531)
 		(width 0.254)
 		(layer "B.Cu")
@@
 	)
 	(segment
-		(start 358.273499 53.1961)
-		(end 358.017091 53.452508)
+		(start 358.273499 51.6086)
+		(end 358.017091 51.865008)
 		(width 0.254)
 		(layer "B.Cu")
@@
 	)
 	(segment
-		(start 359.017091 53.452508)
-		(end 358.760683 53.1961)
+		(start 359.017091 51.865008)
+		(end 358.760683 51.6086)
 		(width 0.254)
 		(layer "B.Cu")
@@
 	)
 	(segment
-		(start 357.017091 54.2481)
+		(start 356.743091 56.0451)
 		(end 357.017091 55.7711)
 		(width 0.254)
@@
 	(segment
 		(start 357.017091 55.7711)
-		(end 356.743091 56.0451)
+		(end 357.017091 52.6606)
 		(width 0.254)
 		(layer "B.Cu")
@@
 	)
 	(segment
-		(start 360.717091 53.562706)
-		(end 359.832985 52.6786)
+		(start 355.817091 52.6606)
+		(end 355.817091 56.4391)
 		(width 0.381)
 		(layer "B.Cu")
@@
 	)
 	(segment
-		(start 355.817091 54.2481)
-		(end 355.817091 56.4391)
+		(start 360.717091 51.975206)
+		(end 359.832985 51.0911)
 		(width 0.381)
 		(layer "B.Cu")
@@
 	)
 	(segment
-		(start 355.817091 53.562706)
-		(end 355.817091 54.2481)
+		(start 355.817091 51.975206)
+		(end 355.817091 52.6606)
 		(width 0.381)
 		(layer "B.Cu")
@@
 	)
 	(segment
-		(start 356.701197 52.6786)
-		(end 355.817091 53.562706)
+		(start 356.701197 51.0911)
+		(end 355.817091 51.975206)
 		(width 0.381)
 		(layer "B.Cu")
@@
 	)
 	(segment
-		(start 360.717091 54.2481)
-		(end 360.717091 53.562706)
+		(start 360.717091 52.6606)
+		(end 360.717091 51.975206)
 		(width 0.381)
 		(layer "B.Cu")
@@
 	)
 	(segment
-		(start 359.832985 52.6786)
-		(end 356.701197 52.6786)
+		(start 359.832985 51.0911)
+		(end 356.701197 51.0911)
 		(width 0.381)
 		(layer "B.Cu")
@@
 	)
 	(segment
+		(start 360.182623 56.055632)
+		(end 360.126623 56.055632)
+		(width 0.254)
+		(layer "B.Cu")
+		(net "Net-(J2-CC2)")
+	)
+	(segment
 		(start 364.109091 55.6641)
 		(end 364.109091 51.6021)
@@
 	)
 	(segment
-		(start 360.182623 56.055632)
-		(end 360.126623 56.055632)
+		(start 360.017091 55.9461)
+		(end 360.017091 52.6606)
 		(width 0.254)
 		(layer "B.Cu")
@@
 		(width 0.254)
 		(layer "B.Cu")
-		(net "Net-(J2-CC2)")
-	)
-	(segment
-		(start 360.017091 55.9461)
-		(end 360.017091 54.2481)
-		(width 0.254)
-		(layer "B.Cu")
