File: keyboard-pcb.kicad_pcb (KiCad board)
At the start: 2 copper layers, 304.8 x 114.3 mm, 359 parts, among them J2 USB_C_Receptacle_USB2.0_16P, U1 STM32F072CBTx, U3 XC6206PxxxMR

Commit message: updates
changed fuse rating from 500mA to 1A, added 470 ohm resistor to start of LED data line, added silkscreen art
Parts:
- added G***: LOGO, LOGO, F.Cu at (158.4, 156.1)
- added G***: LOGO, LOGO, F.Cu at (347.7, 113.4)
- added R6: 470, smd_silkscreen:R_0402_1005Metric, B.Cu at (65.9, 67.1)
- F1: value 500mA -> 1A
Connections:
- LED1 pad 3: LED_in -> /LED Matrix/LED_in
Routing:
- net /LED Matrix/LED_in: track 0.00 -> 4.05 mm
- net LED_in: track 246.9 -> 243.8 mm
- net GND: track 1166.3 -> 1164.9 mm
- net row5: track 307.9 -> 309.3 mm
- net Net-(LED76-DIN): track 67.5 -> 68.6 mm
- net +5V: track 2071.8 -> 2072.5 mm
