File: led-matrix.kicad_sch (KiCad schematic)
At the start: 167 parts

Commit message: assigned footprints
Parts:
- C11, C12, C13, C14, C15, C16, C17, C18, C19, C20, C21, C22, C23, C24, C25, C26, C27, C28, C29, C30, C31, C32, C33, C34, C35, C36, C37, C38, C39, C40, C41, C42, C43, C44, C45, C46, C47, C48, C49, C50, C51, C52, C53, C54, C55, C56, C57, C58, C59, C60, C61, C62, C63, C64, C65, C66, C67, C68, C69, C70, C71, C72, C73, C74, C75, C76, C77, C78, C79, C80, C81, C82, C83, C84, C85, C86, C87, C88, C89, C90, C91, C92, C93: footprint (none) -> Capacitor_SMD:C_0402_1005Metric

Commit message: routed switch matrix
Parts:
- removed D100, D101, D102, D103, D104, D105, D106, D107, D108, D109, D110, D111, D112, D113, D114, D115, D116, D117, D118, D119, D120, D121, D122, D123, D124, D125, D126, D127, D128, D129, D130, D131, D132, D133, D134, D135, D136, D137, D138, D139, D140, D141, D142, D143, D144, D145, D146, D147, D148, D149, D150, D151, D152, D153, D154, D155, D156, D157, D158, D159, D160, D161, D162, D163, D164, D165, D166, D167, D168, D86, D87, D88, D90, D91, D92, D93, D94, D95, D96, D97, D98, D99: SK6812MINI-E, LED_SMD:LED_SK6812MINI-E_3.2x2.8mm_P1.5mm_ReverseMount, symbol LED:SK6812MINI-E
- added C84: 100nF, Capacitor_SMD:C_0402_1005Metric, symbol Device:C_Small
- added LED10, LED11, LED12, LED13, LED14, LED15, LED16, LED17, LED18, LED19, LED2, LED20, LED21, LED22, LED23, LED24, LED25, LED26, LED27, LED28, LED29, LED3, LED30, LED31, LED32, LED33, LED34, LED35, LED36, LED37, LED38, LED39, LED4, LED40, LED41, LED42, LED43, LED44, LED45, LED46, LED47, LED48, LED49, LED50, LED51, LED52, LED53, LED54, LED55, LED56, LED57, LED58, LED59, LED6, LED60, LED61, LED62, LED63, LED64, LED65, LED66, LED67, LED68, LED69, LED7, LED70, LED71, LED72, LED73, LED74, LED75, LED76, LED77, LED78, LED79, LED8, LED80, LED81, LED82, LED83, LED84, LED9: SK6812MINI-E, LED_SMD:LED_SK6812MINI-E_3.2x2.8mm_P1.5mm_ReverseMount, symbol LED:SK6812MINI-E
- renumbered C11 to C1, C20 to C10, C21 to C11, C22 to C12, C23 to C13, C24 to C14, C25 to C15, C26 to C16, C27 to C17, C29 to C18, C31 to C19, C12 to C2, C33 to C20, C35 to C21, C37 to C22, C39 to C23, C41 to C24, C28 to C25, C30 to C26, C32 to C27, C34 to C28, C36 to C29, C13 to C3, C38 to C30, C40 to C31, C42 to C32, C43 to C33, C47 to C34, C51 to C35, C55 to C36, C59 to C37, C63 to C38, C67 to C39, C14 to C4, C71 to C40, C44 to C41, C48 to C42, C52 to C43, C56 to C44, C60 to C45, C64 to C46, C68 to C47, C72 to C48, C45 to C49, C15 to C5, C49 to C50, C53 to C51, C57 to C52, C61 to C53, C65 to C54, C69 to C55, C73 to C56, C46 to C57, C50 to C58, C54 to C59, C16 to C6, C58 to C60, C62 to C61, C66 to C62, C70 to C63, C74 to C64, C75 to C65, C77 to C66, C79 to C67, C81 to C68, C83 to C69, C17 to C7, C85 to C70, C87 to C71, C89 to C72, C76 to C73, C78 to C74, C80 to C75, C82 to C76, C84 to C77, C86 to C78, C88 to C79, C18 to C8, C90 to C80, C91 to C81, C92 to C82, C93 to C83, C19 to C9, D85 to LED1, D89 to LED5
Connections:
- net +3V3 is gone; now on net +5V: C1.1, C10.1, C11.1, C12.1, C13.1, C14.1, C15.1, C16.1, C17.1, C18.1, C19.1, C2.1, C20.1, C21.1, C22.1, C23.1, C24.1, C25.1, C26.1, C27.1, C28.1, C29.1, C3.1, C30.1, C31.1, C32.1, C33.1, C34.1, C35.1, C36.1, C37.1, C38.1, C39.1, C4.1, C40.1, C41.1, C42.1, C43.1, C44.1, C45.1, C46.1, C47.1, C48.1, C49.1, C5.1, C50.1, C51.1, C52.1, C53.1, C54.1, C55.1, C56.1, C57.1, C58.1, C59.1, C6.1, C60.1, C61.1, C62.1, C63.1, C64.1, C65.1, C66.1, C67.1, C68.1, C69.1, C7.1, C70.1, C71.1, C72.1, C73.1, C74.1, C75.1, C76.1, C77.1, C78.1, C79.1, C8.1, C80.1, C81.1, C82.1, C83.1, C9.1
- net +5V: now also C84.1, LED10.3 (VDD), LED11.3 (VDD), LED12.3 (VDD), LED13.3 (VDD), LED14.3 (VDD), LED15.3 (VDD), LED16.3 (VDD), LED17.3 (VDD), LED18.3 (VDD), LED19.3 (VDD), LED2.3 (VDD), LED20.3 (VDD), LED21.3 (VDD), LED22.3 (VDD), LED23.3 (VDD), LED24.3 (VDD), LED25.3 (VDD), LED26.3 (VDD), LED27.3 (VDD), LED28.3 (VDD), LED29.3 (VDD), LED3.3 (VDD), LED30.3 (VDD), LED31.3 (VDD), LED32.3 (VDD), LED33.3 (VDD), LED34.3 (VDD), LED35.3 (VDD), LED36.3 (VDD), LED37.3 (VDD), LED38.3 (VDD), LED39.3 (VDD), LED4.3 (VDD), LED40.3 (VDD), LED41.3 (VDD), LED42.3 (VDD), LED43.3 (VDD), LED44.3 (VDD), LED45.3 (VDD), LED46.3 (VDD), LED47.3 (VDD), LED48.3 (VDD), LED49.3 (VDD), LED50.3 (VDD), LED51.3 (VDD), LED52.3 (VDD), LED53.3 (VDD), LED54.3 (VDD), LED55.3 (VDD), LED56.3 (VDD), LED57.3 (VDD), LED58.3 (VDD), LED59.3 (VDD), LED6.3 (VDD), LED60.3 (VDD), LED61.3 (VDD), LED62.3 (VDD), LED63.3 (VDD), LED64.3 (VDD), LED65.3 (VDD), LED66.3 (VDD), LED67.3 (VDD), LED68.3 (VDD), LED69.3 (VDD), LED7.3 (VDD), LED70.3 (VDD), LED71.3 (VDD), LED72.3 (VDD), LED73.3 (VDD), LED74.3 (VDD), LED75.3 (VDD), LED76.3 (VDD), LED77.3 (VDD), LED78.3 (VDD), LED79.3 (VDD), LED8.3 (VDD), LED80.3 (VDD), LED81.3 (VDD), LED82.3 (VDD), LED83.3 (VDD), LED84.3 (VDD), LED9.3 (VDD)
- net GND: now also C84.2, LED10.1 (VSS), LED11.1 (VSS), LED12.1 (VSS), LED13.1 (VSS), LED14.1 (VSS), LED15.1 (VSS), LED16.1 (VSS), LED17.1 (VSS), LED18.1 (VSS), LED19.1 (VSS), LED2.1 (VSS), LED20.1 (VSS), LED21.1 (VSS), LED22.1 (VSS), LED23.1 (VSS), LED24.1 (VSS), LED25.1 (VSS), LED26.1 (VSS), LED27.1 (VSS), LED28.1 (VSS), LED29.1 (VSS), LED3.1 (VSS), LED30.1 (VSS), LED31.1 (VSS), LED32.1 (VSS), LED33.1 (VSS), LED34.1 (VSS), LED35.1 (VSS), LED36.1 (VSS), LED37.1 (VSS), LED38.1 (VSS), LED39.1 (VSS), LED4.1 (VSS), LED40.1 (VSS), LED41.1 (VSS), LED42.1 (VSS), LED43.1 (VSS), LED44.1 (VSS), LED45.1 (VSS), LED46.1 (VSS), LED47.1 (VSS), LED48.1 (VSS), LED49.1 (VSS), LED50.1 (VSS), LED51.1 (VSS), LED52.1 (VSS), LED53.1 (VSS), LED54.1 (VSS), LED55.1 (VSS), LED56.1 (VSS), LED57.1 (VSS), LED58.1 (VSS), LED59.1 (VSS), LED6.1 (VSS), LED60.1 (VSS), LED61.1 (VSS), LED62.1 (VSS), LED63.1 (VSS), LED64.1 (VSS), LED65.1 (VSS), LED66.1 (VSS), LED67.1 (VSS), LED68.1 (VSS), LED69.1 (VSS), LED7.1 (VSS), LED70.1 (VSS), LED71.1 (VSS), LED72.1 (VSS), LED73.1 (VSS), LED74.1 (VSS), LED75.1 (VSS), LED76.1 (VSS), LED77.1 (VSS), LED78.1 (VSS), LED79.1 (VSS), LED8.1 (VSS), LED80.1 (VSS), LED81.1 (VSS), LED82.1 (VSS), LED83.1 (VSS), LED84.1 (VSS), LED9.1 (VSS)
- net at LED1.4 (DOUT): now also LED2.2 (DIN)
- net at LED5.2 (DIN): now also LED4.4 (DOUT)
- net at LED5.4 (DOUT): now also LED6.2 (DIN)
- new net: LED41.4 (DOUT), LED42.2 (DIN)
- new net: LED42.4 (DOUT), LED43.2 (DIN)
- new net: LED3.4 (DOUT), LED4.2 (DIN)
- new net: LED75.4 (DOUT), LED76.2 (DIN)
- new net: LED76.4 (DOUT), LED77.2 (DIN)
- new net: LED29.4 (DOUT), LED30.2 (DIN)
- new net: LED30.4 (DOUT), LED31.2 (DIN)
- new net: LED78.4 (DOUT), LED79.2 (DIN)
- new net: LED79.4 (DOUT), LED80.2 (DIN)
- new net: LED2.4 (DOUT), LED3.2 (DIN)
- new net: LED62.4 (DOUT), LED63.2 (DIN)
- new net: LED63.4 (DOUT), LED64.2 (DIN)
- new net: LED6.4 (DOUT), LED7.2 (DIN)
- new net: LED7.4 (DOUT), LED8.2 (DIN)
- new net: LED50.4 (DOUT), LED51.2 (DIN)
- new net: LED51.4 (DOUT), LED52.2 (DIN)
- new net: LED25.4 (DOUT), LED26.2 (DIN)
- new net: LED26.4 (DOUT), LED27.2 (DIN)
- new net: LED66.4 (DOUT), LED67.2 (DIN)
- new net: LED67.4 (DOUT), LED68.2 (DIN)
- new net: LED43.4 (DOUT), LED44.2 (DIN)
- new net: LED44.4 (DOUT), LED45.2 (DIN)
- new net: LED82.4 (DOUT), LED83.2 (DIN)
- new net: LED54.4 (DOUT), LED55.2 (DIN)
- new net: LED55.4 (DOUT), LED56.2 (DIN)
- new net: LED21.4 (DOUT), LED22.2 (DIN)
- new net: LED22.4 (DOUT), LED23.2 (DIN)
- new net: LED8.4 (DOUT), LED9.2 (DIN)
- new net: LED35.4 (DOUT), LED36.2 (DIN)
- new net: LED36.4 (DOUT), LED37.2 (DIN)
- new net: LED57.4 (DOUT), LED58.2 (DIN)
- new net: LED58.4 (DOUT), LED59.2 (DIN)
- new net: LED46.4 (DOUT), LED47.2 (DIN)
- new net: LED47.4 (DOUT), LED48.2 (DIN)
- new net: LED61.4 (DOUT), LED62.2 (DIN)
- new net: LED37.4 (DOUT), LED38.2 (DIN)
- new net: LED38.4 (DOUT), LED39.2 (DIN)
- new net: LED59.4 (DOUT), LED60.2 (DIN)
- new net: LED16.2 (DIN), LED84.4 (DOUT)
- new net: LED16.4 (DOUT), LED17.2 (DIN)
- new net: LED52.4 (DOUT), LED53.2 (DIN)
- new net: LED53.4 (DOUT), LED54.2 (DIN)
- new net: LED27.4 (DOUT), LED28.2 (DIN)
- new net: LED28.4 (DOUT), LED29.2 (DIN)
- new net: LED65.4 (DOUT), LED66.2 (DIN)
- new net: LED56.4 (DOUT), LED57.2 (DIN)
- new net: LED17.4 (DOUT), LED18.2 (DIN)
- new net: LED14.4 (DOUT), LED15.2 (DIN)
- new net: LED15.4 (DOUT), LED84.2 (DIN)
- new net: LED23.4 (DOUT), LED24.2 (DIN)
- new net: LED24.4 (DOUT), LED25.2 (DIN)
- new net: LED10.2 (DIN), LED9.4 (DOUT)
- new net: LED10.4 (DOUT), LED11.2 (DIN)
- new net: LED39.4 (DOUT), LED40.2 (DIN)
- new net: LED40.4 (DOUT), LED41.2 (DIN)
- new net: LED11.4 (DOUT), LED12.2 (DIN)
- new net: LED12.4 (DOUT), LED13.2 (DIN)
- new net: LED80.4 (DOUT), LED81.2 (DIN)
- new net: LED81.4 (DOUT), LED82.2 (DIN)
- new net: LED60.4 (DOUT), LED61.2 (DIN)
- new net: LED19.4 (DOUT), LED20.2 (DIN)
- new net: LED20.4 (DOUT), LED21.2 (DIN)
- new net: LED68.4 (DOUT), LED69.2 (DIN)
- new net: LED69.4 (DOUT), LED70.2 (DIN)
- new net: LED72.4 (DOUT), LED73.2 (DIN)
- new net: LED73.4 (DOUT), LED74.2 (DIN)
- new net: LED64.4 (DOUT), LED65.2 (DIN)
- new net: LED70.4 (DOUT), LED71.2 (DIN)
- new net: LED45.4 (DOUT), LED46.2 (DIN)
- new net: LED13.4 (DOUT), LED14.2 (DIN)
- new net: LED48.4 (DOUT), LED49.2 (DIN)
- new net: LED49.4 (DOUT), LED50.2 (DIN)
- new net: LED74.4 (DOUT), LED75.2 (DIN)
- new net: LED33.4 (DOUT), LED34.2 (DIN)
- new net: LED34.4 (DOUT), LED35.2 (DIN)
- new net: LED18.4 (DOUT), LED19.2 (DIN)
- new net: LED32.4 (DOUT), LED33.2 (DIN)
- new net: LED77.4 (DOUT), LED78.2 (DIN)
- new net: LED71.4 (DOUT), LED72.2 (DIN)
- new net: LED31.4 (DOUT), LED32.2 (DIN)
Other:
- moved on the sheet: C81, C82, C83

Commit message: completed pcb design
Parts:
- removed LED1, LED10, LED11, LED12, LED13, LED14, LED15, LED16, LED17, LED18, LED19, LED2, LED20, LED21, LED22, LED23, LED24, LED25, LED26, LED27, LED28, LED29, LED3, LED30, LED31, LED32, LED33, LED34, LED35, LED36, LED37, LED38, LED39, LED4, LED40, LED41, LED42, LED43, LED44, LED45, LED46, LED47, LED48, LED49, LED5, LED50, LED51, LED52, LED53, LED54, LED55, LED56, LED57, LED58, LED59, LED6, LED60, LED61, LED62, LED63, LED64, LED65, LED66, LED67, LED68, LED69, LED7, LED70, LED71, LED72, LED73, LED74, LED75, LED76, LED77, LED78, LED79, LED8, LED80, LED81, LED82, LED83, LED84, LED9: SK6812MINI-E, LED_SMD:LED_SK6812MINI-E_3.2x2.8mm_P1.5mm_ReverseMount, symbol LED:SK6812MINI-E
- added LED1, LED10, LED11, LED12, LED13, LED14, LED15, LED2, LED3, LED31, LED32, LED33, LED34, LED35, LED36, LED37, LED38, LED39, LED4, LED40, LED41, LED42, LED43, LED44, LED45, LED5, LED6, LED60, LED61, LED62, LED63, LED64, LED65, LED66, LED67, LED68, LED69, LED7, LED70, LED71, LED72, LED73, LED8, LED84, LED9: MX_SK6812MINI-E, PCM_marbastlib-mx:LED_MX_6028R-ROT, symbol PCM_marbastlib-mx:MX_SK6812MINI-E
- added LED16, LED17, LED18, LED19, LED20, LED21, LED22, LED23, LED24, LED25, LED26, LED27, LED28, LED29, LED30, LED46, LED47, LED48, LED49, LED50, LED51, LED52, LED53, LED54, LED55, LED56, LED57, LED58, LED59, LED74, LED75, LED76, LED77, LED78, LED79, LED80, LED81, LED82, LED83: MX_SK6812MINI-E, PCM_marbastlib-mx:LED_MX_6028R, symbol PCM_marbastlib-mx:MX_SK6812MINI-E
- C1, C10, C11, C12, C13, C14, C15, C16, C17, C18, C19, C2, C20, C21, C22, C23, C24, C25, C26, C27, C28, C29, C3, C30, C31, C32, C33, C34, C35, C36, C37, C38, C39, C4, C40, C41, C42, C43, C44, C45, C46, C47, C48, C49, C5, C50, C51, C52, C53, C54, C55, C56, C57, C58, C59, C6, C60, C61, C62, C63, C64, C65, C66, C67, C68, C69, C7, C70, C71, C72, C73, C74, C75, C76, C77, C78, C79, C8, C80, C81, C82, C83, C84, C9: footprint Capacitor_SMD:C_0402_1005Metric -> smd_silkscreen:C_0402_1005Metric
Connections:
- net +5V: now also LED1.1 (VDD), LED10.1 (VDD), LED11.1 (VDD), LED12.1 (VDD), LED13.1 (VDD), LED14.1 (VDD), LED15.1 (VDD), LED16.1 (VDD), LED17.1 (VDD), LED18.1 (VDD), LED19.1 (VDD), LED2.1 (VDD), LED20.1 (VDD), LED21.1 (VDD), LED22.1 (VDD), LED23.1 (VDD), LED24.1 (VDD), LED25.1 (VDD), LED26.1 (VDD), LED27.1 (VDD), LED28.1 (VDD), LED29.1 (VDD), LED3.1 (VDD), LED30.1 (VDD), LED31.1 (VDD), LED32.1 (VDD), LED33.1 (VDD), LED34.1 (VDD), LED35.1 (VDD), LED36.1 (VDD), LED37.1 (VDD), LED38.1 (VDD), LED39.1 (VDD), LED4.1 (VDD), LED40.1 (VDD), LED41.1 (VDD), LED42.1 (VDD), LED43.1 (VDD), LED44.1 (VDD), LED45.1 (VDD), LED46.1 (VDD), LED47.1 (VDD), LED48.1 (VDD), LED49.1 (VDD), LED5.1 (VDD), LED50.1 (VDD), LED51.1 (VDD), LED52.1 (VDD), LED53.1 (VDD), LED54.1 (VDD), LED55.1 (VDD), LED56.1 (VDD), LED57.1 (VDD), LED58.1 (VDD), LED59.1 (VDD), LED6.1 (VDD), LED60.1 (VDD), LED61.1 (VDD), LED62.1 (VDD), LED63.1 (VDD), LED64.1 (VDD), LED65.1 (VDD), LED66.1 (VDD), LED67.1 (VDD), LED68.1 (VDD), LED69.1 (VDD), LED7.1 (VDD), LED70.1 (VDD), LED71.1 (VDD), LED72.1 (VDD), LED73.1 (VDD), LED74.1 (VDD), LED75.1 (VDD), LED76.1 (VDD), LED77.1 (VDD), LED78.1 (VDD), LED79.1 (VDD), LED8.1 (VDD), LED80.1 (VDD), LED81.1 (VDD), LED82.1 (VDD), LED83.1 (VDD), LED84.1 (VDD), LED9.1 (VDD)
- net GND: now also LED1.4 (VSS), LED10.4 (VSS), LED11.4 (VSS), LED12.4 (VSS), LED13.4 (VSS), LED14.4 (VSS), LED15.4 (VSS), LED16.4 (VSS), LED17.4 (VSS), LED18.4 (VSS), LED19.4 (VSS), LED2.4 (VSS), LED20.4 (VSS), LED21.4 (VSS), LED22.4 (VSS), LED23.4 (VSS), LED24.4 (VSS), LED25.4 (VSS), LED26.4 (VSS), LED27.4 (VSS), LED28.4 (VSS), LED29.4 (VSS), LED3.4 (VSS), LED30.4 (VSS), LED31.4 (VSS), LED32.4 (VSS), LED33.4 (VSS), LED34.4 (VSS), LED35.4 (VSS), LED36.4 (VSS), LED37.4 (VSS), LED38.4 (VSS), LED39.4 (VSS), LED4.4 (VSS), LED40.4 (VSS), LED41.4 (VSS), LED42.4 (VSS), LED43.4 (VSS), LED44.4 (VSS), LED45.4 (VSS), LED46.4 (VSS), LED47.4 (VSS), LED48.4 (VSS), LED49.4 (VSS), LED5.4 (VSS), LED50.4 (VSS), LED51.4 (VSS), LED52.4 (VSS), LED53.4 (VSS), LED54.4 (VSS), LED55.4 (VSS), LED56.4 (VSS), LED57.4 (VSS), LED58.4 (VSS), LED59.4 (VSS), LED6.4 (VSS), LED60.4 (VSS), LED61.4 (VSS), LED62.4 (VSS), LED63.4 (VSS), LED64.4 (VSS), LED65.4 (VSS), LED66.4 (VSS), LED67.4 (VSS), LED68.4 (VSS), LED69.4 (VSS), LED7.4 (VSS), LED70.4 (VSS), LED71.4 (VSS), LED72.4 (VSS), LED73.4 (VSS), LED74.4 (VSS), LED75.4 (VSS), LED76.4 (VSS), LED77.4 (VSS), LED78.4 (VSS), LED79.4 (VSS), LED8.4 (VSS), LED80.4 (VSS), LED81.4 (VSS), LED82.4 (VSS), LED83.4 (VSS), LED84.4 (VSS), LED9.4 (VSS)
- net LED_in: now also LED1.3 (DIN)
- new net: LED62.2 (DOUT), LED63.3 (DIN)
- new net: LED61.2 (DOUT), LED62.3 (DIN)
- new net: LED15.2 (DOUT), LED84.3 (DIN)
- new net: LED14.2 (DOUT), LED15.3 (DIN)
- new net: LED22.3 (DIN), LED23.2 (DOUT)
- new net: LED23.3 (DIN), LED24.2 (DOUT)
- new net: LED47.3 (DIN), LED48.2 (DOUT)
- new net: LED48.3 (DIN), LED49.2 (DOUT)
- new net: LED16.2 (DOUT), LED31.3 (DIN)
- new net: LED16.3 (DIN), LED17.2 (DOUT)
- new net: LED7.2 (DOUT), LED8.3 (DIN)
- new net: LED6.2 (DOUT), LED7.3 (DIN)
- new net: LED54.3 (DIN), LED55.2 (DOUT)
- new net: LED55.3 (DIN), LED56.2 (DOUT)
- new net: LED80.3 (DIN), LED81.2 (DOUT)
- new net: LED81.3 (DIN), LED82.2 (DOUT)
- new net: LED73.2 (DOUT), LED83.3 (DIN)
- new net: LED72.2 (DOUT), LED73.3 (DIN)
- new net: LED12.2 (DOUT), LED13.3 (DIN)
- new net: LED11.2 (DOUT), LED12.3 (DIN)
- new net: LED56.3 (DIN), LED57.2 (DOUT)
- new net: LED57.3 (DIN), LED58.2 (DOUT)
- new net: LED82.3 (DIN), LED83.2 (DOUT)
- new net: LED21.3 (DIN), LED22.2 (DOUT)
- new net: LED26.3 (DIN), LED27.2 (DOUT)
- new net: LED27.3 (DIN), LED28.2 (DOUT)
- new net: LED28.3 (DIN), LED29.2 (DOUT)
- new net: LED5.2 (DOUT), LED6.3 (DIN)
- new net: LED4.2 (DOUT), LED5.3 (DIN)
- new net: LED17.3 (DIN), LED18.2 (DOUT)
- new net: LED77.3 (DIN), LED78.2 (DOUT)
- new net: LED78.3 (DIN), LED79.2 (DOUT)
- new net: LED71.2 (DOUT), LED72.3 (DIN)
- new net: LED40.2 (DOUT), LED41.3 (DIN)
- new net: LED39.2 (DOUT), LED40.3 (DIN)
- new net: LED8.2 (DOUT), LED9.3 (DIN)
- new net: LED60.2 (DOUT), LED61.3 (DIN)
- new net: LED25.3 (DIN), LED26.2 (DOUT)
- new net: LED10.2 (DOUT), LED11.3 (DIN)
- new net: LED10.3 (DIN), LED9.2 (DOUT)
- new net: LED75.3 (DIN), LED76.2 (DOUT)
- new net: LED76.3 (DIN), LED77.2 (DOUT)
- new net: LED46.2 (DOUT), LED60.3 (DIN)
- new net: LED46.3 (DIN), LED47.2 (DOUT)
- new net: LED13.2 (DOUT), LED14.3 (DIN)
- new net: LED29.3 (DIN), LED30.2 (DOUT)
- new net: LED69.2 (DOUT), LED70.3 (DIN)
- new net: LED68.2 (DOUT), LED69.3 (DIN)
- new net: LED44.2 (DOUT), LED45.3 (DIN)
- new net: LED43.2 (DOUT), LED44.3 (DIN)
- new net: LED49.3 (DIN), LED50.2 (DOUT)
- new net: LED36.2 (DOUT), LED37.3 (DIN)
- new net: LED35.2 (DOUT), LED36.3 (DIN)
- new net: LED74.3 (DIN), LED75.2 (DOUT)
- new net: LED65.2 (DOUT), LED66.3 (DIN)
- new net: LED64.2 (DOUT), LED65.3 (DIN)
- new net: LED66.2 (DOUT), LED67.3 (DIN)
- new net: LED37.2 (DOUT), LED38.3 (DIN)
- new net: LED30.3 (DIN), LED84.2 (DOUT)
- new net: LED79.3 (DIN), LED80.2 (DOUT)
- new net: LED33.2 (DOUT), LED34.3 (DIN)
- new net: LED32.2 (DOUT), LED33.3 (DIN)
- new net: LED58.3 (DIN), LED59.2 (DOUT)
- new net: LED45.2 (DOUT), LED59.3 (DIN)
- new net: LED31.2 (DOUT), LED32.3 (DIN)
- new net: LED38.2 (DOUT), LED39.3 (DIN)
- new net: LED42.2 (DOUT), LED43.3 (DIN)
- new net: LED34.2 (DOUT), LED35.3 (DIN)
- new net: LED20.3 (DIN), LED21.2 (DOUT)
- new net: LED18.3 (DIN), LED19.2 (DOUT)
- new net: LED2.2 (DOUT), LED3.3 (DIN)
- new net: LED1.2 (DOUT), LED2.3 (DIN)
- new net: LED3.2 (DOUT), LED4.3 (DIN)
- new net: LED24.3 (DIN), LED25.2 (DOUT)
- new net: LED63.2 (DOUT), LED64.3 (DIN)
- new net: LED67.2 (DOUT), LED68.3 (DIN)
- new net: LED70.2 (DOUT), LED71.3 (DIN)
- new net: LED50.3 (DIN), LED51.2 (DOUT)
- new net: LED41.2 (DOUT), LED42.3 (DIN)
- new net: LED19.3 (DIN), LED20.2 (DOUT)
- new net: LED53.3 (DIN), LED54.2 (DOUT)
- new net: LED51.3 (DIN), LED52.2 (DOUT)
- new net: LED52.3 (DIN), LED53.2 (DOUT)
