File: keyboard-matrix.kicad_sch (KiCad schematic)
At the start: 0 parts

Commit message: added keyboard switch matrix
Parts:
- added D1, D10, D11, D12, D13, D14, D15, D16, D17, D18, D19, D20, D21, D22, D23, D24, D25, D26, D27, D28, D29, D3, D30, D31, D32, D33, D34, D35, D36, D37, D38, D39, D4, D40, D41, D42, D43, D44, D45, D46, D47, D48, D49, D5, D50, D51, D52, D53, D54, D55, D56, D57, D58, D59, D6, D60, D61, D62, D63, D64, D65, D66, D67, D68, D69, D7, D70, D71, D72, D73, D74, D75, D76, D77, D78, D79, D8, D80, D81, D82, D83, D84, D85, D9: D, symbol Device:D
- added MX1: HS_esc, PCM_marbastlib-mx:SW_MX_HS_CPG151101S11_1u, symbol PCM_marbastlib-mx:MX_SW_HS_CPG151101S11
- added MX10: HS_f9, PCM_marbastlib-mx:SW_MX_HS_CPG151101S11_1u, symbol PCM_marbastlib-mx:MX_SW_HS_CPG151101S11
- added MX11: HS_f10, PCM_marbastlib-mx:SW_MX_HS_CPG151101S11_1u, symbol PCM_marbastlib-mx:MX_SW_HS_CPG151101S11
- added MX12: HS_f11, PCM_marbastlib-mx:SW_MX_HS_CPG151101S11_1u, symbol PCM_marbastlib-mx:MX_SW_HS_CPG151101S11
- added MX13: HS_f12, PCM_marbastlib-mx:SW_MX_HS_CPG151101S11_1u, symbol PCM_marbastlib-mx:MX_SW_HS_CPG151101S11
- added MX14: HS_ins, PCM_marbastlib-mx:SW_MX_HS_CPG151101S11_1u, symbol PCM_marbastlib-mx:MX_SW_HS_CPG151101S11
- added MX15: HS_del, PCM_marbastlib-mx:SW_MX_HS_CPG151101S11_1u, symbol PCM_marbastlib-mx:MX_SW_HS_CPG151101S11
- added MX16: HS_extra, PCM_marbastlib-mx:SW_MX_HS_CPG151101S11_1u, symbol PCM_marbastlib-mx:MX_SW_HS_CPG151101S11
- added MX17: HS_~, PCM_marbastlib-mx:SW_MX_HS_CPG151101S11_1u, symbol PCM_marbastlib-mx:MX_SW_HS_CPG151101S11
- added MX18: HS_#1, PCM_marbastlib-mx:SW_MX_HS_CPG151101S11_1u, symbol PCM_marbastlib-mx:MX_SW_HS_CPG151101S11
- added MX19: HS_#2, PCM_marbastlib-mx:SW_MX_HS_CPG151101S11_1u, symbol PCM_marbastlib-mx:MX_SW_HS_CPG151101S11
- added MX2: HS_f1, PCM_marbastlib-mx:SW_MX_HS_CPG151101S11_1u, symbol PCM_marbastlib-mx:MX_SW_HS_CPG151101S11
- added MX20: HS_#3, PCM_marbastlib-mx:SW_MX_HS_CPG151101S11_1u, symbol PCM_marbastlib-mx:MX_SW_HS_CPG151101S11
- added MX21: HS_#4, PCM_marbastlib-mx:SW_MX_HS_CPG151101S11_1u, symbol PCM_marbastlib-mx:MX_SW_HS_CPG151101S11
- added MX22: HS_#5, PCM_marbastlib-mx:SW_MX_HS_CPG151101S11_1u, symbol PCM_marbastlib-mx:MX_SW_HS_CPG151101S11
- added MX23: HS_#6, PCM_marbastlib-mx:SW_MX_HS_CPG151101S11_1u, symbol PCM_marbastlib-mx:MX_SW_HS_CPG151101S11
- added MX24: HS_#7, PCM_marbastlib-mx:SW_MX_HS_CPG151101S11_1u, symbol PCM_marbastlib-mx:MX_SW_HS_CPG151101S11
- added MX25: HS_#8, PCM_marbastlib-mx:SW_MX_HS_CPG151101S11_1u, symbol PCM_marbastlib-mx:MX_SW_HS_CPG151101S11
- added MX26: HS_#9, PCM_marbastlib-mx:SW_MX_HS_CPG151101S11_1u, symbol PCM_marbastlib-mx:MX_SW_HS_CPG151101S11
- added MX27: HS_#0, PCM_marbastlib-mx:SW_MX_HS_CPG151101S11_1u, symbol PCM_marbastlib-mx:MX_SW_HS_CPG151101S11
- added MX28: HS_-, PCM_marbastlib-mx:SW_MX_HS_CPG151101S11_1u, symbol PCM_marbastlib-mx:MX_SW_HS_CPG151101S11
- added MX29: HS_=, PCM_marbastlib-mx:SW_MX_HS_CPG151101S11_1u, symbol PCM_marbastlib-mx:MX_SW_HS_CPG151101S11
- added MX3: HS_f2, PCM_marbastlib-mx:SW_MX_HS_CPG151101S11_1u, symbol PCM_marbastlib-mx:MX_SW_HS_CPG151101S11
- added MX30: HS_back, PCM_marbastlib-mx:SW_MX_HS_CPG151101S11_1u, symbol PCM_marbastlib-mx:MX_SW_HS_CPG151101S11
- added MX31: HS_home, PCM_marbastlib-mx:SW_MX_HS_CPG151101S11_1u, symbol PCM_marbastlib-mx:MX_SW_HS_CPG151101S11
- added MX32: HS_tab, PCM_marbastlib-mx:SW_MX_HS_CPG151101S11_1u, symbol PCM_marbastlib-mx:MX_SW_HS_CPG151101S11
- added MX33: HS_Q, PCM_marbastlib-mx:SW_MX_HS_CPG151101S11_1u, symbol PCM_marbastlib-mx:MX_SW_HS_CPG151101S11
- added MX34: HS_W, PCM_marbastlib-mx:SW_MX_HS_CPG151101S11_1u, symbol PCM_marbastlib-mx:MX_SW_HS_CPG151101S11
- added MX35: HS_E, PCM_marbastlib-mx:SW_MX_HS_CPG151101S11_1u, symbol PCM_marbastlib-mx:MX_SW_HS_CPG151101S11
- added MX36: HS_R, PCM_marbastlib-mx:SW_MX_HS_CPG151101S11_1u, symbol PCM_marbastlib-mx:MX_SW_HS_CPG151101S11
- added MX37: HS_T, PCM_marbastlib-mx:SW_MX_HS_CPG151101S11_1u, symbol PCM_marbastlib-mx:MX_SW_HS_CPG151101S11
- added MX38: HS_Y, PCM_marbastlib-mx:SW_MX_HS_CPG151101S11_1u, symbol PCM_marbastlib-mx:MX_SW_HS_CPG151101S11
- added MX39: HS_U, PCM_marbastlib-mx:SW_MX_HS_CPG151101S11_1u, symbol PCM_marbastlib-mx:MX_SW_HS_CPG151101S11
- added MX4: HS_f3, PCM_marbastlib-mx:SW_MX_HS_CPG151101S11_1u, symbol PCM_marbastlib-mx:MX_SW_HS_CPG151101S11
- added MX40: HS_I, PCM_marbastlib-mx:SW_MX_HS_CPG151101S11_1u, symbol PCM_marbastlib-mx:MX_SW_HS_CPG151101S11
- added MX41: HS_O, PCM_marbastlib-mx:SW_MX_HS_CPG151101S11_1u, symbol PCM_marbastlib-mx:MX_SW_HS_CPG151101S11
- added MX42: HS_P, PCM_marbastlib-mx:SW_MX_HS_CPG151101S11_1u, symbol PCM_marbastlib-mx:MX_SW_HS_CPG151101S11
- added MX43: HS_[, PCM_marbastlib-mx:SW_MX_HS_CPG151101S11_1u, symbol PCM_marbastlib-mx:MX_SW_HS_CPG151101S11
- added MX44: HS_], PCM_marbastlib-mx:SW_MX_HS_CPG151101S11_1u, symbol PCM_marbastlib-mx:MX_SW_HS_CPG151101S11
- added MX45: HS_\, PCM_marbastlib-mx:SW_MX_HS_CPG151101S11_1u, symbol PCM_marbastlib-mx:MX_SW_HS_CPG151101S11
- added MX46: HS_end, PCM_marbastlib-mx:SW_MX_HS_CPG151101S11_1u, symbol PCM_marbastlib-mx:MX_SW_HS_CPG151101S11
- added MX47: HS_caps, PCM_marbastlib-mx:SW_MX_HS_CPG151101S11_1u, symbol PCM_marbastlib-mx:MX_SW_HS_CPG151101S11
- added MX48: HS_A, PCM_marbastlib-mx:SW_MX_HS_CPG151101S11_1u, symbol PCM_marbastlib-mx:MX_SW_HS_CPG151101S11
- added MX49: HS_S, PCM_marbastlib-mx:SW_MX_HS_CPG151101S11_1u, symbol PCM_marbastlib-mx:MX_SW_HS_CPG151101S11
- added MX5: HS_f4, PCM_marbastlib-mx:SW_MX_HS_CPG151101S11_1u, symbol PCM_marbastlib-mx:MX_SW_HS_CPG151101S11
- added MX50: HS_D, PCM_marbastlib-mx:SW_MX_HS_CPG151101S11_1u, symbol PCM_marbastlib-mx:MX_SW_HS_CPG151101S11
- added MX51: HS_F, PCM_marbastlib-mx:SW_MX_HS_CPG151101S11_1u, symbol PCM_marbastlib-mx:MX_SW_HS_CPG151101S11
- added MX52: HS_G, PCM_marbastlib-mx:SW_MX_HS_CPG151101S11_1u, symbol PCM_marbastlib-mx:MX_SW_HS_CPG151101S11
- added MX53: HS_H, PCM_marbastlib-mx:SW_MX_HS_CPG151101S11_1u, symbol PCM_marbastlib-mx:MX_SW_HS_CPG151101S11
- added MX54: HS_J, PCM_marbastlib-mx:SW_MX_HS_CPG151101S11_1u, symbol PCM_marbastlib-mx:MX_SW_HS_CPG151101S11
- added MX55: HS_K, PCM_marbastlib-mx:SW_MX_HS_CPG151101S11_1u, symbol PCM_marbastlib-mx:MX_SW_HS_CPG151101S11
- added MX56: HS_L, PCM_marbastlib-mx:SW_MX_HS_CPG151101S11_1u, symbol PCM_marbastlib-mx:MX_SW_HS_CPG151101S11
- added MX57: HS_;, PCM_marbastlib-mx:SW_MX_HS_CPG151101S11_1u, symbol PCM_marbastlib-mx:MX_SW_HS_CPG151101S11
- added MX58: HS_', PCM_marbastlib-mx:SW_MX_HS_CPG151101S11_1u, symbol PCM_marbastlib-mx:MX_SW_HS_CPG151101S11
- added MX59: HS_enter, PCM_marbastlib-mx:SW_MX_HS_CPG151101S11_1u, symbol PCM_marbastlib-mx:MX_SW_HS_CPG151101S11
- added MX6: HS_f5, PCM_marbastlib-mx:SW_MX_HS_CPG151101S11_1u, symbol PCM_marbastlib-mx:MX_SW_HS_CPG151101S11
- added MX60: HS_pgup, PCM_marbastlib-mx:SW_MX_HS_CPG151101S11_1u, symbol PCM_marbastlib-mx:MX_SW_HS_CPG151101S11
- added MX61: HS_Lshift, PCM_marbastlib-mx:SW_MX_HS_CPG151101S11_1u, symbol PCM_marbastlib-mx:MX_SW_HS_CPG151101S11
- added MX62: HS_Z, PCM_marbastlib-mx:SW_MX_HS_CPG151101S11_1u, symbol PCM_marbastlib-mx:MX_SW_HS_CPG151101S11
- added MX63: HS_X, PCM_marbastlib-mx:SW_MX_HS_CPG151101S11_1u, symbol PCM_marbastlib-mx:MX_SW_HS_CPG151101S11
- added MX64: HS_C, PCM_marbastlib-mx:SW_MX_HS_CPG151101S11_1u, symbol PCM_marbastlib-mx:MX_SW_HS_CPG151101S11
- added MX65: HS_V, PCM_marbastlib-mx:SW_MX_HS_CPG151101S11_1u, symbol PCM_marbastlib-mx:MX_SW_HS_CPG151101S11
- added MX66: HS_B, PCM_marbastlib-mx:SW_MX_HS_CPG151101S11_1u, symbol PCM_marbastlib-mx:MX_SW_HS_CPG151101S11
- added MX67: HS_N, PCM_marbastlib-mx:SW_MX_HS_CPG151101S11_1u, symbol PCM_marbastlib-mx:MX_SW_HS_CPG151101S11
- added MX68: HS_M, PCM_marbastlib-mx:SW_MX_HS_CPG151101S11_1u, symbol PCM_marbastlib-mx:MX_SW_HS_CPG151101S11
- added MX69: HS_<, PCM_marbastlib-mx:SW_MX_HS_CPG151101S11_1u, symbol PCM_marbastlib-mx:MX_SW_HS_CPG151101S11
- added MX7: HS_f6, PCM_marbastlib-mx:SW_MX_HS_CPG151101S11_1u, symbol PCM_marbastlib-mx:MX_SW_HS_CPG151101S11
- added MX70: HS_>, PCM_marbastlib-mx:SW_MX_HS_CPG151101S11_1u, symbol PCM_marbastlib-mx:MX_SW_HS_CPG151101S11
- added MX71: HS_/, PCM_marbastlib-mx:SW_MX_HS_CPG151101S11_1u, symbol PCM_marbastlib-mx:MX_SW_HS_CPG151101S11
- added MX72: HS_Rshift, PCM_marbastlib-mx:SW_MX_HS_CPG151101S11_1u, symbol PCM_marbastlib-mx:MX_SW_HS_CPG151101S11
- added MX73: HS_up, PCM_marbastlib-mx:SW_MX_HS_CPG151101S11_1u, symbol PCM_marbastlib-mx:MX_SW_HS_CPG151101S11
- added MX74: HS_pgdn, PCM_marbastlib-mx:SW_MX_HS_CPG151101S11_1u, symbol PCM_marbastlib-mx:MX_SW_HS_CPG151101S11
- added MX75: HS_Lctrl, PCM_marbastlib-mx:SW_MX_HS_CPG151101S11_1u, symbol PCM_marbastlib-mx:MX_SW_HS_CPG151101S11
- added MX76: HS_win, PCM_marbastlib-mx:SW_MX_HS_CPG151101S11_1u, symbol PCM_marbastlib-mx:MX_SW_HS_CPG151101S11
- added MX77: HS_Lalt, PCM_marbastlib-mx:SW_MX_HS_CPG151101S11_1u, symbol PCM_marbastlib-mx:MX_SW_HS_CPG151101S11
- added MX78: HS_space, PCM_marbastlib-mx:SW_MX_HS_CPG151101S11_1u, symbol PCM_marbastlib-mx:MX_SW_HS_CPG151101S11
- added MX79: HS_Ralt, PCM_marbastlib-mx:SW_MX_HS_CPG151101S11_1u, symbol PCM_marbastlib-mx:MX_SW_HS_CPG151101S11
- added MX8: HS_f7, PCM_marbastlib-mx:SW_MX_HS_CPG151101S11_1u, symbol PCM_marbastlib-mx:MX_SW_HS_CPG151101S11
- added MX80: HS_fn, PCM_marbastlib-mx:SW_MX_HS_CPG151101S11_1u, symbol PCM_marbastlib-mx:MX_SW_HS_CPG151101S11
- added MX81: HS_Rctrl, PCM_marbastlib-mx:SW_MX_HS_CPG151101S11_1u, symbol PCM_marbastlib-mx:MX_SW_HS_CPG151101S11
- added MX82: HS_left, PCM_marbastlib-mx:SW_MX_HS_CPG151101S11_1u, symbol PCM_marbastlib-mx:MX_SW_HS_CPG151101S11
- added MX83: HS_down, PCM_marbastlib-mx:SW_MX_HS_CPG151101S11_1u, symbol PCM_marbastlib-mx:MX_SW_HS_CPG151101S11
- added MX84: HS_right, PCM_marbastlib-mx:SW_MX_HS_CPG151101S11_1u, symbol PCM_marbastlib-mx:MX_SW_HS_CPG151101S11
- added MX9: HS_f8, PCM_marbastlib-mx:SW_MX_HS_CPG151101S11_1u, symbol PCM_marbastlib-mx:MX_SW_HS_CPG151101S11
Connections:
- new net: D4.2 (A), MX3.2
- new net: D6.2 (A), MX5.2
- new net: D65.2 (A), MX64.2
- new net: D25.2 (A), MX24.2
- new net: D85.2 (A), MX84.2
- new net: D17.2 (A), MX16.2
- new net: D42.2 (A), MX41.2
- new net: D12.2 (A), MX11.2
- new net: D63.2 (A), MX62.2
- new net: D5.2 (A), MX4.2
- new net: D59.2 (A), MX58.2
- new net: D64.2 (A), MX63.2
- new net: D79.2 (A), MX78.2
- new net: D55.2 (A), MX54.2
- new net: D28.2 (A), MX27.2
- new net: D44.2 (A), MX43.2
- new net: D67.2 (A), MX66.2
- new net: D47.2 (A), MX46.2
- new net: D15.2 (A), MX14.2
- new net: D57.2 (A), MX56.2
- new net: D58.2 (A), MX57.2
- new net: D30.2 (A), MX29.2
- new net: D21.2 (A), MX20.2
- new net: D36.2 (A), MX35.2
- new net: D46.2 (A), MX45.2
- new net: D20.2 (A), MX19.2
- new net: D3.2 (A), MX2.2
- new net: D50.2 (A), MX49.2
- new net: D9.2 (A), MX8.2
- new net: D84.2 (A), MX83.2
- new net: D33.2 (A), MX32.2
- new net: D19.2 (A), MX18.2
- new net: D56.2 (A), MX55.2
- new net: D78.2 (A), MX77.2
- new net: D82.2 (A), MX81.2
- new net: D1.2 (A), MX1.2
- new net: D77.2 (A), MX76.2
- new net: D23.2 (A), MX22.2
- new net: D81.2 (A), MX80.2
- new net: D51.2 (A), MX50.2
- new net: D16.2 (A), MX15.2
- new net: D53.2 (A), MX52.2
- new net: D35.2 (A), MX34.2
- new net: D14.2 (A), MX13.2
- new net: D11.2 (A), MX10.2
- new net: D54.2 (A), MX53.2
- new net: D39.2 (A), MX38.2
- new net: D72.2 (A), MX71.2
- new net: D37.2 (A), MX36.2
- new net: D8.2 (A), MX7.2
- new net: D34.2 (A), MX33.2
- new net: D76.2 (A), MX75.2
- new net: D52.2 (A), MX51.2
- new net: D29.2 (A), MX28.2
- new net: D18.2 (A), MX17.2
- new net: D45.2 (A), MX44.2
- new net: D61.2 (A), MX60.2
- new net: D48.2 (A), MX47.2
- new net: D10.2 (A), MX9.2
- new net: D60.2 (A), MX59.2
- new net: D43.2 (A), MX42.2
- new net: D22.2 (A), MX21.2
- new net: D24.2 (A), MX23.2
- new net: D73.2 (A), MX72.2
- new net: D62.2 (A), MX61.2
- new net: D74.2 (A), MX73.2
- new net: D40.2 (A), MX39.2
- new net: D70.2 (A), MX69.2
- new net: D13.2 (A), MX12.2
- new net: D38.2 (A), MX37.2
- new net: D69.2 (A), MX68.2
- new net: D26.2 (A), MX25.2
- new net: D75.2 (A), MX74.2
- new net: D68.2 (A), MX67.2
- new net: D7.2 (A), MX6.2
- new net: D31.2 (A), MX30.2
- new net: D80.2 (A), MX79.2
- new net: D49.2 (A), MX48.2
- new net: D66.2 (A), MX65.2
- new net: D83.2 (A), MX82.2
- new net: D32.2 (A), MX31.2
- new net: D27.2 (A), MX26.2
- new net: D71.2 (A), MX70.2
- new net: D41.2 (A), MX40.2
- new net col0: MX1.1, MX17.1, MX32.1, MX47.1, MX61.1, MX75.1
- new net col1: MX18.1, MX2.1, MX33.1, MX48.1, MX62.1, MX76.1
- new net col10: MX11.1, MX27.1, MX42.1, MX57.1, MX71.1, MX81.1
- new net col11: MX12.1, MX28.1, MX43.1, MX58.1, MX72.1, MX82.1
- new net col12: MX13.1, MX29.1, MX44.1
- new net col13: MX14.1, MX30.1, MX45.1, MX59.1, MX73.1, MX83.1
- new net col14: MX15.1, MX31.1, MX46.1, MX60.1, MX74.1, MX84.1
- new net col15: MX16.1
- new net col2: MX19.1, MX3.1, MX34.1, MX49.1, MX63.1, MX77.1
- new net col3: MX20.1, MX35.1, MX4.1, MX50.1, MX64.1
- new net col4: MX21.1, MX36.1, MX5.1, MX51.1, MX65.1
- new net col5: MX22.1, MX37.1, MX52.1, MX6.1, MX66.1, MX78.1
- new net col6: MX23.1, MX38.1, MX53.1, MX67.1, MX7.1
- new net col7: MX24.1, MX39.1, MX54.1, MX68.1, MX8.1
- new net col8: MX25.1, MX40.1, MX55.1, MX69.1, MX79.1, MX9.1
- new net col9: MX10.1, MX26.1, MX41.1, MX56.1, MX70.1, MX80.1
- new net row0: D1.1 (K), D10.1 (K), D11.1 (K), D12.1 (K), D13.1 (K), D14.1 (K), D15.1 (K), D16.1 (K), D17.1 (K), D3.1 (K), D4.1 (K), D5.1 (K), D6.1 (K), D7.1 (K), D8.1 (K), D9.1 (K)
- new net row1: D18.1 (K), D19.1 (K), D20.1 (K), D21.1 (K), D22.1 (K), D23.1 (K), D24.1 (K), D25.1 (K), D26.1 (K), D27.1 (K), D28.1 (K), D29.1 (K), D30.1 (K), D31.1 (K), D32.1 (K)
- new net row2: D33.1 (K), D34.1 (K), D35.1 (K), D36.1 (K), D37.1 (K), D38.1 (K), D39.1 (K), D40.1 (K), D41.1 (K), D42.1 (K), D43.1 (K), D44.1 (K), D45.1 (K), D46.1 (K), D47.1 (K)
- new net row3: D48.1 (K), D49.1 (K), D50.1 (K), D51.1 (K), D52.1 (K), D53.1 (K), D54.1 (K), D55.1 (K), D56.1 (K), D57.1 (K), D58.1 (K), D59.1 (K), D60.1 (K), D61.1 (K)
- new net row4: D62.1 (K), D63.1 (K), D64.1 (K), D65.1 (K), D66.1 (K), D67.1 (K), D68.1 (K), D69.1 (K), D70.1 (K), D71.1 (K), D72.1 (K), D73.1 (K), D74.1 (K), D75.1 (K)
- new net row5: D76.1 (K), D77.1 (K), D78.1 (K), D79.1 (K), D80.1 (K), D81.1 (K), D82.1 (K), D83.1 (K), D84.1 (K), D85.1 (K)

Commit message: added led matrix for backlight
Parts:
- removed D17: D, symbol Device:D
- removed MX16: HS_extra, PCM_marbastlib-mx:SW_MX_HS_CPG151101S11_1u, symbol PCM_marbastlib-mx:MX_SW_HS_CPG151101S11
- renumbered D18 to D17, D19 to D18, D20 to D19, D21 to D20, D22 to D21, D23 to D22, D24 to D23, D25 to D24, D26 to D25, D27 to D26, D28 to D27, D29 to D28, D30 to D29, D31 to D30, D32 to D31, D33 to D32, D34 to D33, D35 to D34, D36 to D35, D37 to D36, D38 to D37, D39 to D38, D40 to D39, D41 to D40, D42 to D41, D43 to D42, D44 to D43, D45 to D44, D46 to D45, D47 to D46, D48 to D47, D49 to D48, D50 to D49, D51 to D50, D52 to D51, D53 to D52, D54 to D53, D55 to D54, D56 to D55, D57 to D56, D58 to D57, D59 to D58, D60 to D59, D61 to D60, D62 to D61, D63 to D62, D64 to D63, D65 to D64, D66 to D65, D67 to D66, D68 to D67, D69 to D68, D70 to D69, D71 to D70, D72 to D71, D73 to D72, D74 to D73, D75 to D74, D76 to D75, D77 to D76, D78 to D77, D79 to D78, D80 to D79, D81 to D80, D82 to D81, D83 to D82, D84 to D83, D85 to D84, MX17 to MX16, MX18 to MX17, MX19 to MX18, MX20 to MX19, MX21 to MX20, MX22 to MX21, MX23 to MX22, MX24 to MX23, MX25 to MX24, MX26 to MX25, MX27 to MX26, MX28 to MX27, MX29 to MX28, MX30 to MX29, MX31 to MX30, MX32 to MX31, MX33 to MX32, MX34 to MX33, MX35 to MX34, MX36 to MX35, MX37 to MX36, MX38 to MX37, MX39 to MX38, MX40 to MX39, MX41 to MX40, MX42 to MX41, MX43 to MX42, MX44 to MX43, MX45 to MX44, MX46 to MX45, MX47 to MX46, MX48 to MX47, MX49 to MX48, MX50 to MX49, MX51 to MX50, MX52 to MX51, MX53 to MX52, MX54 to MX53, MX55 to MX54, MX56 to MX55, MX57 to MX56, MX58 to MX57, MX59 to MX58, MX60 to MX59, MX61 to MX60, MX62 to MX61, MX63 to MX62, MX64 to MX63, MX65 to MX64, MX66 to MX65, MX67 to MX66, MX68 to MX67, MX69 to MX68, MX70 to MX69, MX71 to MX70, MX72 to MX71, MX73 to MX72, MX74 to MX73, MX75 to MX74, MX76 to MX75, MX77 to MX76, MX78 to MX77, MX79 to MX78, MX80 to MX79, MX81 to MX80, MX82 to MX81, MX83 to MX82, MX84 to MX83

Commit message: assigned footprints
Parts:
- D10, D11, D12, D13, D14, D15, D16, D17, D18, D19, D20, D21, D22, D23, D24, D25, D26, D27, D28, D29, D3, D30, D31, D32, D33, D34, D35, D36, D37, D38, D39, D4, D40, D41, D42, D43, D44, D45, D46, D47, D48, D49, D5, D50, D51, D52, D53, D54, D55, D56, D57, D58, D59, D6, D60, D61, D62, D63, D64, D65, D66, D67, D68, D69, D7, D70, D71, D72, D73, D74, D75, D76, D77, D78, D79, D8, D80, D81, D82, D83, D84, D9: footprint (none) -> Diode_SMD:D_SOD-123
- D2: renamed from D1; footprint (none) -> Diode_SMD:D_SOD-123

Commit message: routed switch matrix
Parts:
- added S1, S2: MX_stab, PCM_marbastlib-mx:STAB_MX_2.25u, symbol PCM_marbastlib-mx:MX_stab
- added S3: MX_stab, PCM_marbastlib-mx:STAB_MX_6.25u, symbol PCM_marbastlib-mx:MX_stab
- MX31: footprint PCM_marbastlib-mx:SW_MX_HS_CPG151101S11_1u -> PCM_marbastlib-mx:SW_MX_HS_CPG151101S11_1.5u
- MX46: footprint PCM_marbastlib-mx:SW_MX_HS_CPG151101S11_1u -> PCM_marbastlib-mx:SW_MX_HS_CPG151101S11_1.75u
- MX74, MX75, MX76: footprint PCM_marbastlib-mx:SW_MX_HS_CPG151101S11_1u -> PCM_marbastlib-mx:SW_MX_HS_CPG151101S11_1.25u
Changed lines of the file:
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@@
 			)
 		)
-		(property "Footprint" "PCM_marbastlib-mx:SW_MX_HS_CPG151101S11_1u"
+		(property "Footprint" "PCM_marbastlib-mx:SW_MX_HS_CPG151101S11_1.5u"
 			(at 55.245 84.455 0)
 			(hide yes)
@@
 			)
 		)
-		(property "Footprint" "PCM_marbastlib-mx:SW_MX_HS_CPG151101S11_1u"
+		(property "Footprint" "PCM_marbastlib-mx:SW_MX_HS_CPG151101S11_1.25u"
 			(at 67.945 151.13 0)
 			(hide yes)
@@
 			)
 		)
-		(property "Footprint" "PCM_marbastlib-mx:SW_MX_HS_CPG151101S11_1u"
+		(property "Footprint" "PCM_marbastlib-mx:SW_MX_HS_CPG151101S11_1.25u"
 			(at 55.245 151.13 0)
 			(hide yes)
@@
 			)
 		)
-		(property "Footprint" "PCM_marbastlib-mx:SW_MX_HS_CPG151101S11_1u"
+		(property "Footprint" "PCM_marbastlib-mx:SW_MX_HS_CPG151101S11_1.75u"
 			(at 55.245 106.68 0)
 			(hide yes)
@@
 	)
 	(symbol
+		(lib_id "PCM_marbastlib-mx:MX_stab")
+		(at 208.915 106.68 0)
+		(unit 1)
+		(body_style 1)
+		(exclude_from_sim no)
+		(in_bom yes)
+		(on_board yes)
+		(in_pos_files yes)
+		(dnp no)
+		(property "Reference" "S1"
+			(at 205.359 100.33 0)
+			(show_name no)
+			(do_not_autoplace no)
+			(effects
+				(font
+					(size 1.27 1.27)
+				)
+				(justify left)
+			)
+		)
+		(property "Value" "MX_stab"
+			(at 205.359 102.87 0)
+			(show_name no)
+			(do_not_autoplace no)
+			(effects
+				(font
+					(size 1.27 1.27)
+				)
+				(justify left)
+			)
+		)
+		(property "Footprint" "PCM_marbastlib-mx:STAB_MX_2.25u"
+			(at 208.915 106.68 0)
+			(hide yes)
+			(show_name no)
+			(do_not_autoplace no)
+			(effects
+				(font
+					(size 1.27 1.27)
+				)
+			)
+		)
+		(property "Datasheet" ""
+			(at 208.915 106.68 0)
+			(hide yes)
+			(show_name no)
+			(do_not_autoplace no)
+			(effects
+				(font
+					(size 1.27 1.27)
+				)
+			)
+		)
+		(property "Description" "Cherry MX-style stabilizer"
+			(at 208.915 106.68 0)
+			(hide yes)
+			(show_name no)
+			(do_not_autoplace no)
+			(effects
+				(font
+					(size 1.27 1.27)
+				)
+			)
+		)
+		(instances
+			(project "keyboard-pcb"
+				(path "/a41dad29-4328-40a3-b427-6ea31b74fde8/bc94a4ef-73e7-4422-8e97-826f4e66b418"
+					(reference "S1")
+					(unit 1)
+				)
+			)
+		)
+	)
+	(symbol
 		(lib_id "Device:D")
 		(at 197.485 113.03 90)
@@
 			)
 		)
-		(property "Footprint" "PCM_marbastlib-mx:SW_MX_HS_CPG151101S11_1u"
+		(property "Footprint" "PCM_marbastlib-mx:SW_MX_HS_CPG151101S11_1.25u"
 			(at 80.645 151.13 0)
 			(hide yes)
@@
 	)
 	(symbol
+		(lib_id "PCM_marbastlib-mx:MX_stab")
+		(at 39.37 130.175 0)
+		(unit 1)
+		(body_style 1)
+		(exclude_from_sim no)
+		(in_bom yes)
+		(on_board yes)
+		(in_pos_files yes)
+		(dnp no)
+		(property "Reference" "S2"
+			(at 35.56 123.698 0)
+			(show_name no)
+			(do_not_autoplace no)
+			(effects
+				(font
+					(size 1.27 1.27)
+				)
+				(justify left)
+			)
+		)
+		(property "Value" "MX_stab"
+			(at 35.56 126.238 0)
+			(show_name no)
+			(do_not_autoplace no)
+			(effects
+				(font
+					(size 1.27 1.27)
+				)
+				(justify left)
+			)
+		)
+		(property "Footprint" "PCM_marbastlib-mx:STAB_MX_2.25u"
+			(at 39.37 130.175 0)
+			(hide yes)
+			(show_name no)
+			(do_not_autoplace no)
+			(effects
+				(font
+					(size 1.27 1.27)
+				)
+			)
+		)
+		(property "Datasheet" ""
+			(at 39.37 130.175 0)
+			(hide yes)
+			(show_name no)
+			(do_not_autoplace no)
+			(effects
+				(font
+					(size 1.27 1.27)
+				)
+			)
+		)
+		(property "Description" "Cherry MX-style stabilizer"
+			(at 39.37 130.175 0)
+			(hide yes)
+			(show_name no)
+			(do_not_autoplace no)
+			(effects
+				(font
+					(size 1.27 1.27)
+				)
+			)
+		)
+		(instances
+			(project "keyboard-pcb"
+				(path "/a41dad29-4328-40a3-b427-6ea31b74fde8/bc94a4ef-73e7-4422-8e97-826f4e66b418"
+					(reference "S2")
+					(unit 1)
+				)
+			)
+		)
+	)
+	(symbol
 		(lib_id "Device:D")
 		(at 57.785 113.03 90)
@@
 					(unit 1)
 				)
+			)
+		)
+	)
+	(symbol
+		(lib_id "PCM_marbastlib-mx:MX_stab")
+		(at 139.065 151.13 0)
+		(unit 1)
+		(body_style 1)
+		(exclude_from_sim no)
+		(in_bom yes)
+		(on_board yes)
+		(in_pos_files yes)
+		(dnp no)
+		(fields_autoplaced yes)
+		(property "Reference" "S3"
+			(at 144.78 149.7329 0)
+			(show_name no)
+			(do_not_autoplace no)
+			(effects
+				(font
+					(size 1.27 1.27)
+				)
+				(justify left)
+			)
+		)
+		(property "Value" "MX_stab"
+			(at 144.78 152.2729 0)
+			(show_name no)
+			(do_not_autoplace no)
+			(effects
+				(font
+					(size 1.27 1.27)
+				)
+				(justify left)
+			)
+		)
+		(property "Footprint" "PCM_marbastlib-mx:STAB_MX_6.25u"
+			(at 139.065 151.13 0)
+			(hide yes)
+			(show_name no)
+			(do_not_autoplace no)
+			(effects
+				(font
+					(size 1.27 1.27)
+				)
+			)
+		)
+		(property "Datasheet" ""
+			(at 139.065 151.13 0)
+			(hide yes)
+			(show_name no)
+			(do_not_autoplace no)
+			(effects
+				(font
+					(size 1.27 1.27)
+				)
+			)
+		)
+		(property "Description" "Cherry MX-style stabilizer"
+			(at 139.065 151.13 0)
+			(hide yes)
+			(show_name no)
+			(do_not_autoplace no)
+			(effects
+				(font
+					(size 1.27 1.27)
+				)
+			)
+		)
+		(instances
+			(project "keyboard-pcb"
+				(path "/a41dad29-4328-40a3-b427-6ea31b74fde8/bc94a4ef-73e7-4422-8e97-826f4e66b418"
+					(reference "S3")
+					(unit 1)
+				)

Commit message: completed pcb design
Parts:
- removed S1, S2: MX_stab, PCM_marbastlib-mx:STAB_MX_2.25u, symbol PCM_marbastlib-mx:MX_stab
- removed S3: MX_stab, PCM_marbastlib-mx:STAB_MX_6.25u, symbol PCM_marbastlib-mx:MX_stab
- MX1, MX10, MX11, MX12, MX13, MX14, MX15, MX16, MX17, MX18, MX19, MX2, MX20, MX21, MX22, MX23, MX24, MX25, MX26, MX27, MX28, MX29, MX3, MX30, MX32, MX33, MX34, MX35, MX36, MX37, MX38, MX39, MX4, MX40, MX41, MX42, MX43, MX44, MX45, MX47, MX48, MX49, MX5, MX50, MX51, MX52, MX53, MX54, MX55, MX56, MX57, MX59, MX6, MX61, MX62, MX63, MX64, MX65, MX66, MX67, MX68, MX69, MX7, MX70, MX71, MX72, MX73, MX78, MX79, MX8, MX80, MX81, MX82, MX83, MX9: footprint PCM_marbastlib-mx:SW_MX_HS_CPG151101S11_1u -> MX_Hotswap:MX-Hotswap-1U
- MX31: footprint PCM_marbastlib-mx:SW_MX_HS_CPG151101S11_1.5u -> MX_Hotswap:MX-Hotswap-1.5U
- MX46: footprint PCM_marbastlib-mx:SW_MX_HS_CPG151101S11_1.75u -> MX_Hotswap:MX-Hotswap-1.75U
- MX58, MX60: footprint PCM_marbastlib-mx:SW_MX_HS_CPG151101S11_1u -> MX_Hotswap:MX-Hotswap-2.25U
- MX74, MX75, MX76: footprint PCM_marbastlib-mx:SW_MX_HS_CPG151101S11_1.25u -> MX_Hotswap:MX-Hotswap-1.25U
- MX77: footprint PCM_marbastlib-mx:SW_MX_HS_CPG151101S11_1u -> MX_Hotswap:MX-Hotswap-6.25U

Commit message: revised layout for more compact size
Parts:
- MX77: footprint MX_Hotswap:MX-Hotswap-6.25U -> MX_Hotswap:MX-Hotswap-6.25U-ReversedStabilizers
Changed lines of the file:
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@@
 			)
 		)
-		(property "Footprint" "MX_Hotswap:MX-Hotswap-6.25U"
+		(property "Footprint" "MX_Hotswap:MX-Hotswap-6.25U-ReversedStabilizers"
 			(at 118.745 151.13 0)
 			(hide yes)

Commit message: updated layout
added 2u stabs for backspace, moved usb and mounting hole for clearance
Parts:
- MX29: footprint MX_Hotswap:MX-Hotswap-1U -> MX_Hotswap:MX-Hotswap-2U
Changed lines of the file:
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@@
 			)
 		)
-		(property "Footprint" "MX_Hotswap:MX-Hotswap-1U"
+		(property "Footprint" "MX_Hotswap:MX-Hotswap-2U"
 			(at 220.345 62.23 0)
 			(hide yes)
